File: pcb/bloomer.kicad_pcb (KiCad board)
At the start: 2 copper layers, 322.7 x 132.7 mm, 188 parts, among them U1 ItsyBitsy

Commit message: Rename Ergo87 to Bloomer and update readme
Other:
- board text added: "Bloomer"
- board text added: "By: CozyKeys"
- board text removed: "By: Paul Ewing"
- board text removed: "Ergo87"
Changed lines of the file:
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@@
     (pad 4 smd rect (at 1.65 -2.4 90) (size 1.4 1.8) (layers Back B.Paste B.Mask))
   )
-  (gr_text "By: Paul Ewing" (at 212.09 31.75) (layer B.SilkS)
+  (gr_text "By: CozyKeys" (at 212.09 31.75) (layer B.SilkS)
     (effects (font (size 1.27 1.524) (thickness 0.3048)) (justify mirror))
   )
-  (gr_text Ergo87 (at 212.725 27.305) (layer B.SilkS)
+  (gr_text Bloomer (at 212.725 27.305) (layer B.SilkS)
     (effects (font (size 4.064 3.048) (thickness 0.3048)) (justify mirror))
   )

Commit message: Finish up rev3
Parts:
- removed B1: VAL**, B3F-10XX
- added ?: , Sparkfun-Aesthetics:OSHW-LOGO-M, B.Cu at (74.4, 141.6)
- added ?: , Sparkfun-Aesthetics:OSHW-LOGO-M, F.Cu at (275.6, 141.6)
- added D3:6: , DIODE, F.Cu at (138.7, 95.7)
- added D3:7: , DIODE, F.Cu at (175.0, 135.1)
- added D3:8: , DIODE, F.Cu at (211.3, 95.7)
- added G***: LOGO, myparts:qmk-badge, F.Cu at (284.5, 147.3)
- added G***: LOGO, myparts:qmk-badge, B.Cu at (65.5, 147.3)
- added HOLE_M3: VAL**, HOLE_M3, F.Cu at (21.6, 27.8)
- added HOLE_M3: VAL**, HOLE_M3, F.Cu at (198.5, 111.5)
- added HOLE_M3: VAL**, HOLE_M3, F.Cu at (155.0, 27.8)
- added HOLE_M3: VAL**, HOLE_M3, F.Cu at (195.0, 27.8)
- added HOLE_M3: VAL**, HOLE_M3, F.Cu at (155.0, 60.8)
- added HOLE_M3: VAL**, HOLE_M3, F.Cu at (195.0, 60.8)
- added HOLE_M3: VAL**, HOLE_M3, F.Cu at (328.4, 27.8)
- added HOLE_M3: VAL**, HOLE_M3, F.Cu at (328.4, 140.5)
- added HOLE_M3: VAL**, HOLE_M3, F.Cu at (21.6, 140.5)
- added HOLE_M3: VAL**, HOLE_M3, F.Cu at (151.5, 111.5)
- added SW3:6: , MX_SWITCH, F.Cu at (138.7, 104.7)
- added SW3:7: , MX_SWITCH, F.Cu at (175.0, 144.1)
- added SW3:8: , MX_SWITCH, F.Cu at (211.3, 104.7)
- ItsyBitsy 32u4: renamed from U1
- SW0:0, SW0:1, SW0:10, SW0:11, SW0:12, SW0:13, SW0:14, SW0:2, SW0:3, SW0:4, SW0:5, SW0:6, SW0:7, SW0:8, SW0:9, SW1:0, SW1:1, SW1:10, SW1:11, SW1:12, SW1:13, SW1:14, SW1:2, SW1:3, SW1:4, SW1:5, SW1:6, SW1:7, SW1:8, SW1:9, SW2:0, SW2:1, SW2:10, SW2:11, SW2:12, SW2:13, SW2:14, SW2:2, SW2:3, SW2:4, SW2:5, SW2:6, SW2:7, SW2:8, SW2:9, SW3:0, SW3:1, SW3:10, SW3:11, SW3:12, SW3:13, SW3:14, SW3:2, SW3:3, SW3:4, SW3:5, SW3:9, SW4:0, SW4:1, SW4:10, SW4:11, SW4:12, SW4:13, SW4:14, SW4:2, SW4:3, SW4:4, SW4:5, SW4:6, SW4:7, SW4:8, SW4:9, SW5:0, SW5:1, SW5:10, SW5:11, SW5:12, SW5:13, SW5:14, SW5:2, SW5:3, SW5:4, SW5:5, SW5:6, SW5:7, SW5:8, SW5:9: footprint MX_FLIP -> MX_SWITCH
- moved D0:7 92.7 mm to (155.9, 116.0)
- moved SW0:7 92.6 mm to (155.9, 125.0)
- moved SW1:7 82.8 mm to (155.9, 144.1)
- moved D1:7 76.9 mm to (155.9, 135.1), turned to 0 degrees
- moved SW0:6 48.4 mm to (165.5, 86.9)
- moved SW0:8 48.4 mm to (184.5, 86.9)
- moved D0:6 42.7 mm to (165.5, 77.9), turned to 0 degrees
- moved D0:8 42.7 mm to (184.5, 77.9), turned to 0 degrees
- moved SW2:7 42.5 mm to (175.0, 125.0)
- moved SW1:6 38.7 mm to (165.5, 106.0)
- moved SW1:8 38.7 mm to (184.5, 106.0)
- moved D2:7 34.7 mm to (175.0, 116.0), turned to 0 degrees
- moved D1:8 34.0 mm to (184.5, 97.0), turned to 0 degrees
- moved D4:6 30.2 mm to (135.4, 114.5), turned to 350 degrees
- moved D1:6 28.5 mm to (165.5, 97.0), turned to 0 degrees
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Connections:
- net N-5V-0 renamed 5V
- ItsyBitsy 32u4 pad 1: N-RST -> (no net)
- ItsyBitsy 32u4 pad 32: N-GND-1 -> (no net)
- ItsyBitsy 32u4 pad 4: N-GND-0 -> GND
- RGB0 pad 1: N-GND-1 -> GND
- RGB1 pad 1: N-GND-1 -> GND
- RGB10 pad 1: N-GND-1 -> GND
- RGB11 pad 1: N-GND-1 -> GND
- RGB2 pad 1: N-GND-1 -> GND
- RGB3 pad 1: N-GND-1 -> GND
- RGB4 pad 1: N-GND-1 -> GND
- RGB5 pad 1: N-GND-1 -> GND
- RGB6 pad 1: N-GND-1 -> GND
- RGB7 pad 1: N-GND-1 -> GND
- RGB8 pad 1: N-GND-1 -> GND
- RGB9 pad 1: N-GND-1 -> GND
Routing:
- net N-GND-1: track 931.7 -> 0.00 mm, vias 14 -> 0
- net GND: track 0.00 -> 824.1 mm, vias 0 -> 8
- net N-RST: track 100.6 -> 0.00 mm, vias 3 -> 0
- net N-row-5: track 579.2 -> 480.8 mm, vias 1 -> 2
- net N-GND-0: track 91.4 -> 0.00 mm, vias 3 -> 0
- net N-col-7: track 113.5 -> 177.4 mm, vias 0 -> 2
- net N-col-14: track 235.7 -> 293.5 mm, vias 0 -> 2
- net N-col-11: track 186.3 -> 238.0 mm
- net N-row-1: track 383.2 -> 432.3 mm, vias 1 -> 2
- net N-col-12: track 207.4 -> 254.1 mm, vias 0 -> 2
- net N-col-13: track 224.6 -> 271.1 mm, vias 0 -> 2
- net N-col-9: track 171.9 -> 217.2 mm
- net N-RGB-D11: track 103.6 -> 141.7 mm, vias 2 -> 0
- net N-RGB-D1: track 107.9 -> 144.5 mm, vias 2 -> 0
- net N-col-6: track 141.7 -> 172.6 mm
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Other:
- board size 322.7 x 132.7 mm -> 326.7 x 132.7 mm
- board text added: "CozyKeys Bloomer"
- board text added: "Designed by Paul Ewing"
- board text added: "Open Hardware"
- board text added: "https://github.com/cozykeys/bloomer"
- board text removed: "Bloomer"
- board text removed: "By: CozyKeys"
- board text removed: "RST"

Commit message: Add reset switch to PCB
Parts:
- added RESET: VAL**, B3F-10XX, B.Cu at (175.0, 65.0)
Connections:
- ItsyBitsy 32u4 pad 1: (no net) -> RST
Routing:
- net RST: track 0.00 -> 65.3 mm, vias 0 -> 3
- net GND: track 824.1 -> 882.7 mm, vias 8 -> 10
- net N-col-7: track 177.4 -> 184.3 mm
- net N-row-5: track 480.8 -> 485.6 mm
Changed lines of the file:
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@@
     (thickness 1.6002)
     (drawings 16)
-    (tracks 1488)
+    (tracks 1518)
     (zones 0)
-    (modules 207)
-    (nets 126)
+    (modules 208)
+    (nets 127)
   )
   (page A4)
@@
   (net 124 N-RGB-D10)
   (net 125 N-RGB-D11)
+  (net 126 RST)
   (net_class Default "This is the default net class."
     (clearance 0.254)
@@
     (add_net N-row-4)
     (add_net N-row-5)
+    (add_net RST)
   )
   (module MX_SWITCH (layer Front)
@@
     (fp_line (start -17.78 6.35) (end -15.24 6.35) (layer F.SilkS) (width 0.381))
     (fp_line (start -15.24 6.35) (end -15.24 8.89) (layer F.SilkS) (width 0.381))
-    (pad 1 thru_hole rect (at -16.51 7.62) (size 1.7526 1.7526) (drill 1.0922) (layers *.Cu *.SilkS *.Mask))
+    (pad 1 thru_hole rect (at -16.51 7.62) (size 1.7526 1.7526) (drill 1.0922) (layers *.Cu *.SilkS *.Mask)
+      (net 126 RST))
     (pad 2 thru_hole circle (at -13.97 7.62) (size 1.7526 1.7526) (drill 1.0922) (layers *.Cu *.SilkS *.Mask)
       (net 113 5V))
@@
     (pad 99 smd rect (at 1.6637 0.000002 10) (size 0.8382 0.8382) (layers Back B.Paste B.Mask))
   )
+  (module B3F-10XX (layer Back)
+    (at 175 65)
+    (descr "Tactile switch - SPST - 6mm")
+    (tags "tactile switch")
+    (fp_text reference RESET (at 0 5) (layer B.SilkS)
+      (effects (font (size 1 1) (thickness 0.18)) (justify bottom mirror))
+    )
+    (fp_text value VAL** (at 0 -4.3) (layer B.SilkS) hide
+      (effects (font (size 1 1) (thickness 0.15)) (justify mirror))
+    )
+    (fp_line (start -3.5 3.5) (end 3.5 3.5) (layer B.CrtYd) (width 0.05))
+    (fp_line (start 3.5 3.5) (end 3.5 -3.5) (layer B.CrtYd) (width 0.05))
+    (fp_line (start 3.5 -3.5) (end -3.5 -3.5) (layer B.CrtYd) (width 0.05))
+    (fp_line (start -3.5 -3.5) (end -3.5 3.5) (layer B.CrtYd) (width 0.05))
+    (fp_line (start -3 -1.25) (end -3 1.25) (layer B.SilkS) (width 0.18))
+    (fp_line (start -2.5 -3) (end 2.5 -3) (layer B.SilkS) (width 0.18))
+    (fp_line (start -2.5 3) (end 2.5 3) (layer B.SilkS) (width 0.18))
+    (fp_line (start 3 -1.25) (end 3 1.25) (layer B.SilkS) (width 0.18))
+    (fp_circle (center 0 0) (end 1.75 0) (layer B.SilkS) (width 0.18))
+    (fp_line (start -0.635 0) (end 0.635 0) (layer B.SilkS) (width 0.18))
+    (fp_line (start 0 0.635) (end 0 -0.635) (layer B.SilkS) (width 0.18))
+    (pad 1 thru_hole circle (at -3.25 -2.25) (size 1.6 1.6) (drill 1) (layers *.Cu *.Mask))
+    (pad 1 thru_hole circle (at 3.25 -2.25) (size 1.6 1.6) (drill 1) (layers *.Cu *.Mask)
+      (net 126 RST))
+    (pad 2 thru_hole circle (at 3.25 2.25) (size 1.6 1.6) (drill 1) (layers *.Cu *.Mask)
+      (net 112 GND))
+    (pad 2 thru_hole circle (at -3.25 2.25) (size 1.6 1.6) (drill 1) (layers *.Cu *.Mask))
+  )
   (module WS2812B (layer Back)
     (at 226 21.28 270)
@@
   (segment (start 202.565 127) (end 202.565 116.205) (width 0.2032) (layer Back) (net 6))
   (via (at 198.12 104.775) (size 0.889) (drill 0.635) (layers Front Back) (net 6))
-  (segment (start 164.465 47.625) (end 165.1 46.99) (width 0.2032) (layer Back) (net 6))
-  (segment (start 164.465 59.69) (end 164.465 47.625) (width 0.2032) (layer Back) (net 6))
-  (segment (start 174.625 69.85) (end 164.465 59.69) (width 0.2032) (layer Back) (net 6))
-  (segment (start 198.12 74.295) (end 198.285101 74.129899) (width 0.2032) (layer Back) (net 6))
-  (segment (start 198.12 104.775) (end 198.12 74.295) (width 0.2032) (layer Back) (net 6))
-  (segment (start 198.285101 74.129899) (end 198.285101 73.494899) (width 0.2032) (layer Back) (net 6))
-  (segment (start 165.1 46.99) (end 167.38 46.99) (width 0.2032) (layer Back) (net 6))
-  (segment (start 197.485 69.85) (end 174.625 69.85) (width 0.2032) (layer Back) (net 6))
-  (segment (start 198.285101 73.494899) (end 199.39 72.39) (width 0.2032) (layer Back) (net 6))
-  (segment (start 199.39 72.39) (end 199.39 71.755) (width 0.2032) (layer Back) (net 6))
-  (segment (start 199.39 71.755) (end 197.485 69.85) (width 0.2032) (layer Back) (net 6))
   (segment (start 202.565 109.22) (end 198.12 104.775) (width 0.2032) (layer Front) (net 6))
   (segment (start 202.565 116.205) (end 202.565 109.22) (width 0.2032) (layer Front) (net 6))
+  (segment (start 198.285101 74.129899) (end 198.12 74.295) (width 0.2032) (layer Back) (net 6))
+  (segment (start 199.39 72.39) (end 198.285101 73.494899) (width 0.2032) (layer Back) (net 6))
+  (segment (start 199.39 71.755) (end 199.39 72.39) (width 0.2032) (layer Back) (net 6))
+  (segment (start 198.12 74.295) (end 198.12 104.775) (width 0.2032) (layer Back) (net 6))
+  (segment (start 165.1 46.99) (end 164.465 47.625) (width 0.2032) (layer Back) (net 6))
+  (segment (start 198.285101 73.494899) (end 198.285101 74.129899) (width 0.2032) (layer Back) (net 6))
+  (segment (start 167.38 46.99) (end 165.1 46.99) (width 0.2032) (layer Back) (net 6))
+  (segment (start 166.37 69.85) (end 197.485 69.85) (width 0.2032) (layer Back) (net 6))
+  (segment (start 164.465 47.625) (end 164.465 67.945) (width 0.2032) (layer Back) (net 6))
+  (segment (start 164.465 67.945) (end 166.37 69.85) (width 0.2032) (layer Back) (net 6))
+  (segment (start 197.485 69.85) (end 199.39 71.755) (width 0.2032) (layer Back) (net 6))
   (segment (start 33.242949 37.925989) (end 29.934949 41.233989) (width 0.2032) (layer Front) (net 7))
   (segment (start 29.934949 56.685989) (end 26.626949 59.993989) (width 0.2032) (layer Front) (net 7))
@@
   (via (at 173.99 95.885) (size 0.889) (drill 0.635) (layers Front Back) (net 14))
   (segment (start 173.99 109.855) (end 173.99 95.885) (width 0.2032) (layer Back) (net 14))
-  (segment (start 175 69.475) (end 175 52.07) (width 0.2032) (layer Front) (net 14))
-  (segment (start 173.99 95.885) (end 173.99 70.485) (width 0.2032) (layer Front) (net 14))
-  (segment (start 173.99 70.485) (end 175 69.475) (width 0.2032) (layer Front) (net 14))
+  (segment (start 175 54.61) (end 175 52.07) (width 0.2032) (layer Front) (net 14))
+  (segment (start 169.545 54.61) (end 175 54.61) (width 0.2032) (layer Front) (net 14))
+  (segment (start 169.545 68.58) (end 169.545 54.61) (width 0.2032) (layer Front) (net 14))
+  (segment (start 173.99 73.025) (end 169.545 68.58) (width 0.2032) (layer Front) (net 14))
+  (segment (start 173.99 95.885) (end 173.99 73.025) (width 0.2032) (layer Front) (net 14))
   (segment (start 180.715 84.384) (end 182.174 84.384) (width 0.2032) (layer Front) (net 15))
   (segment (start 182.174 84.384) (end 182.738 83.82) (width 0.2032) (layer Front) (net 15))
@@
   (segment (start 121.53 22.86) (end 121.6 22.93) (width 0.2032) (layer Back) (net 112))
   (segment (start 114.935 22.86) (end 121.53 22.86) (width 0.2032) (layer Back) (net 112))
+  (segment (start 178.25 67.25) (end 179.765 67.25) (width 0.2032) (layer Back) (net 112))
+  (segment (start 179.765 67.25) (end 180.975 66.04) (width 0.2032) (layer Back) (net 112))
+  (segment (start 180.975 66.04) (end 180.975 60.325) (width 0.2032) (layer Back) (net 112))
+  (segment (start 180.975 60.325) (end 180.34 59.69) (width 0.2032) (layer Back) (net 112))
+  (segment (start 180.34 59.69) (end 179.705 59.055) (width 0.2032) (layer Back) (net 112))
+  (via (at 165.735 59.055) (size 0.889) (drill 0.635) (layers Front Back) (net 112))
+  (segment (start 179.705 59.055) (end 165.735 59.055) (width 0.2032) (layer Back) (net 112))
+  (segment (start 165.735 59.055) (end 165.1 58.42) (width 0.2032) (layer Front) (net 112))
+  (segment (start 165.1 58.42) (end 164.465 57.785) (width 0.2032) (layer Front) (net 112))
+  (via (at 164.465 45.72) (size 0.889) (drill 0.635) (layers Front Back) (net 112))
+  (segment (start 164.465 57.785) (end 164.465 45.72) (width 0.2032) (layer Front) (net 112))
+  (segment (start 164.465 45.72) (end 164.465 27.305) (width 0.2032) (layer Back) (net 112))
+  (segment (start 165.1 27.305) (end 165.735 26.67) (width 0.2032) (layer Back) (net 112))
+  (segment (start 164.465 27.305) (end 165.1 27.305) (width 0.2032) (layer Back) (net 112))
   (segment (start 165.735 21.59) (end 167.38 21.59) (width 0.2032) (layer Back) (net 113))
   (segment (start 126.4 19.63) (end 163.775 19.63) (width 0.2032) (layer Back) (net 113))
@@
   (segment (start 119.9168 19.05) (end 120.4968 19.63) (width 0.2032) (layer Back) (net 125))
   (segment (start 23.495 19.05) (end 119.9168 19.05) (width 0.2032) (layer Back) (net 125))
+  (segment (start 178.25 62.75) (end 179.82 62.75) (width 0.2032) (layer Back) (net 126))
+  (segment (start 179.82 62.75) (end 180.34 62.23) (width 0.2032) (layer Back) (net 126))
+  (segment (start 180.34 62.23) (end 180.34 60.96) (width 0.2032) (layer Back) (net 126))
+  (via (at 165.735 60.325) (size 0.889) (drill 0.635) (layers Front Back) (net 126))
+  (segment (start 180.34 60.96) (end 179.705 60.325) (width 0.2032) (layer Back) (net 126))
+  (segment (start 179.705 60.325) (end 165.735 60.325) (width 0.2032) (layer Back) (net 126))
+  (via (at 163.195 60.325) (size 0.889) (drill 0.635) (layers Front Back) (net 126))
+  (segment (start 165.735 60.325) (end 163.195 60.325) (width 0.2032) (layer Front) (net 126))
+  (segment (start 163.195 60.325) (end 163.195 26.67) (width 0.2032) (layer Back) (net 126))
+  (via (at 163.195 26.035) (size 0.889) (drill 0.635) (layers Front Back) (net 126))
+  (segment (start 163.195 26.67) (end 163.195 26.035) (width 0.2032) (layer Back) (net 126))
+  (segment (start 163.195 26.035) (end 163.195 20.955) (width 0.2032) (layer Front) (net 126))
+  (segment (start 165.1 19.05) (end 167.38 19.05) (width 0.2032) (layer Front) (net 126))
+  (segment (start 163.195 20.955) (end 165.1 19.05) (width 0.2032) (layer Front) (net 126))
 )

Commit message: Reorganize files pre-merge
Parts:
- removed ? (x2): , Sparkfun-Aesthetics:OSHW-LOGO-M
- removed D3:6, D3:7, D3:8: , DIODE
- removed G*** (x2): LOGO, myparts:qmk-badge
- removed HOLE_M3 (x10): VAL**, HOLE_M3
- removed RESET: VAL**, B3F-10XX
- removed SW3:6, SW3:7, SW3:8: , MX_SWITCH
- added B1: VAL**, B3F-10XX, B.Cu at (175.0, 98.0)
- SW0:0, SW0:1, SW0:10, SW0:11, SW0:12, SW0:13, SW0:14, SW0:2, SW0:3, SW0:4, SW0:5, SW0:6, SW0:7, SW0:8, SW0:9, SW1:0, SW1:1, SW1:10, SW1:11, SW1:12, SW1:13, SW1:14, SW1:2, SW1:3, SW1:4, SW1:5, SW1:6, SW1:7, SW1:8, SW1:9, SW2:0, SW2:1, SW2:10, SW2:11, SW2:12, SW2:13, SW2:14, SW2:2, SW2:3, SW2:4, SW2:5, SW2:6, SW2:7, SW2:8, SW2:9, SW3:0, SW3:1, SW3:10, SW3:11, SW3:12, SW3:13, SW3:14, SW3:2, SW3:3, SW3:4, SW3:5, SW3:9, SW4:0, SW4:1, SW4:10, SW4:11, SW4:12, SW4:13, SW4:14, SW4:2, SW4:3, SW4:4, SW4:5, SW4:6, SW4:7, SW4:8, SW4:9, SW5:0, SW5:1, SW5:10, SW5:11, SW5:12, SW5:13, SW5:14, SW5:2, SW5:3, SW5:4, SW5:5, SW5:6, SW5:7, SW5:8, SW5:9: footprint MX_SWITCH -> MX_FLIP
- U1: renamed from ItsyBitsy 32u4
- moved D0:7 92.7 mm to (175.3, 25.4)
- moved SW0:7 92.6 mm to (175.0, 34.4)
- moved SW1:7 82.8 mm to (175.0, 63.5)
- moved D1:7 76.9 mm to (184.0, 63.5), turned to 90 degrees
- moved SW0:6 48.4 mm to (155.9, 39.4)
- moved SW0:8 48.4 mm to (194.1, 39.4)
- moved D0:6 42.7 mm to (146.9, 39.4), turned to 90 degrees
- moved D0:8 42.7 mm to (203.1, 39.4), turned to 90 degrees
- moved SW2:7 42.5 mm to (175.0, 82.5)
- moved SW1:6 38.7 mm to (155.9, 68.5)
- moved SW1:8 38.7 mm to (194.1, 68.5)
- moved D2:7 34.7 mm to (184.0, 82.5), turned to 90 degrees
- moved D1:8 34.0 mm to (203.1, 68.5), turned to 90 degrees
- moved D4:6 30.2 mm to (164.9, 120.6), turned to 90 degrees
- moved D1:6 28.5 mm to (164.9, 68.5), turned to 90 degrees
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Connections:
- net 5V renamed N-5V-0
- RGB0 pad 1: GND -> N-GND-1
- RGB1 pad 1: GND -> N-GND-1
- RGB10 pad 1: GND -> N-GND-1
- RGB11 pad 1: GND -> N-GND-1
- RGB2 pad 1: GND -> N-GND-1
- RGB3 pad 1: GND -> N-GND-1
- RGB4 pad 1: GND -> N-GND-1
- RGB5 pad 1: GND -> N-GND-1
- RGB6 pad 1: GND -> N-GND-1
- RGB7 pad 1: GND -> N-GND-1
- RGB8 pad 1: GND -> N-GND-1
- RGB9 pad 1: GND -> N-GND-1
- U1 pad 1: RST -> N-RST
- U1 pad 32: (no net) -> N-GND-1
- U1 pad 4: GND -> N-GND-0
Routing:
- net N-GND-1: track 0.00 -> 931.7 mm, vias 0 -> 14
- net GND: track 882.7 -> 0.00 mm, vias 10 -> 0
- net N-RST: track 0.00 -> 100.6 mm, vias 0 -> 3
- net N-row-5: track 485.6 -> 579.2 mm, vias 2 -> 1
- net N-GND-0: track 0.00 -> 91.4 mm, vias 0 -> 3
- net N-col-7: track 184.3 -> 113.5 mm, vias 2 -> 0
- net RST: track 65.3 -> 0.00 mm, vias 3 -> 0
- net N-col-14: track 293.5 -> 235.7 mm, vias 2 -> 0
- net N-col-11: track 238.0 -> 186.3 mm
- net N-row-1: track 432.3 -> 383.2 mm, vias 2 -> 1
- net N-col-12: track 254.1 -> 207.4 mm, vias 2 -> 0
- net N-col-13: track 271.1 -> 224.6 mm, vias 2 -> 0
- net N-col-9: track 217.2 -> 171.9 mm
- net N-RGB-D11: track 141.7 -> 103.6 mm, vias 0 -> 2
- net N-RGB-D1: track 144.5 -> 107.9 mm, vias 0 -> 2
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Other:
- board size 326.7 x 132.7 mm -> 322.7 x 132.7 mm
- board text added: "Bloomer"
- board text added: "By: CozyKeys"
- board text added: "RST"
- board text removed: "CozyKeys Bloomer"
- board text removed: "Designed by Paul Ewing"
- board text removed: "Open Hardware"
- board text removed: "https://github.com/cozykeys/bloomer"
