File: pcb/bloomer.kicad_pcb (KiCad board)
At the start: 2 copper layers, 322.7 x 132.7 mm, 188 parts, among them U1 ItsyBitsy

Commit message: Progress
Parts:
- removed B1: VAL**, B3F-10XX
- removed D0:0, D0:1, D0:10, D0:11, D0:12, D0:13, D0:14, D0:2, D0:3, D0:4, D0:5, D0:6, D0:7, D0:8, D0:9, D1:0, D1:1, D1:10, D1:11, D1:12, D1:13, D1:14, D1:2, D1:3, D1:4, D1:5, D1:6, D1:7, D1:8, D1:9, D2:0, D2:1, D2:10, D2:11, D2:12, D2:13, D2:14, D2:2, D2:3, D2:4, D2:5, D2:6, D2:7, D2:8, D2:9, D3:0, D3:1, D3:10, D3:11, D3:12, D3:13, D3:14, D3:2, D3:3, D3:4, D3:5, D3:9, D4:0, D4:1, D4:10, D4:11, D4:12, D4:13, D4:14, D4:2, D4:3, D4:4, D4:5, D4:6, D4:7, D4:8, D4:9, D5:0, D5:1, D5:10, D5:11, D5:12, D5:13, D5:14, D5:2, D5:3, D5:4, D5:5, D5:6, D5:7, D5:8, D5:9: , DIODE
- removed SW0:0, SW0:1, SW0:10, SW0:11, SW0:12, SW0:13, SW0:14, SW0:2, SW0:3, SW0:4, SW0:5, SW0:6, SW0:7, SW0:8, SW0:9, SW1:0, SW1:1, SW1:10, SW1:11, SW1:12, SW1:13, SW1:14, SW1:2, SW1:3, SW1:4, SW1:5, SW1:6, SW1:7, SW1:8, SW1:9, SW2:0, SW2:1, SW2:10, SW2:11, SW2:12, SW2:13, SW2:14, SW2:2, SW2:3, SW2:4, SW2:5, SW2:6, SW2:7, SW2:8, SW2:9, SW3:0, SW3:1, SW3:10, SW3:11, SW3:12, SW3:13, SW3:14, SW3:2, SW3:3, SW3:4, SW3:5, SW3:9, SW4:0, SW4:1, SW4:10, SW4:11, SW4:12, SW4:13, SW4:14, SW4:2, SW4:3, SW4:4, SW4:5, SW4:6, SW4:7, SW4:8, SW4:9, SW5:0, SW5:1, SW5:10, SW5:11, SW5:12, SW5:13, SW5:14, SW5:2, SW5:3, SW5:4, SW5:5, SW5:6, SW5:7, SW5:8, SW5:9: , MX_FLIP
- added ?: , MX, F.Cu at (35.1, 25.6)
- added ?: , MX, F.Cu at (221.7, 45.1)
- added ?: , MX, F.Cu at (239.6, 36.9)
- added ?: , MX, F.Cu at (257.3, 27.7)
- added ?: , MX, F.Cu at (276.9, 29.3)
- added ?: , MX, F.Cu at (296.2, 28.9)
- added ?: , MX, F.Cu at (314.9, 25.6)
- added ?: , MX, F.Cu at (31.7, 44.4)
- added ?: , MX, F.Cu at (50.5, 47.7)
- added ?: , MX, F.Cu at (69.8, 48.1)
- added ?: , MX, F.Cu at (89.4, 46.4)
- added ?: , MX, F.Cu at (53.8, 28.9)
- added ?: , MX, F.Cu at (107.1, 55.7)
- added ?: , MX, F.Cu at (125.0, 63.9)
- added ?: , MX, F.Cu at (155.9, 87.0)
- added ?: , MX, F.Cu at (175.0, 87.0)
- added ?: , MX, F.Cu at (194.1, 87.0)
- added ?: , MX, F.Cu at (225.0, 63.9)
- added ?: , MX, F.Cu at (242.9, 55.7)
- added ?: , MX, F.Cu at (260.6, 46.4)
- added ?: , MX, F.Cu at (280.2, 48.1)
- added ?: , MX, F.Cu at (299.5, 47.7)
- added ?: , MX, F.Cu at (73.1, 29.3)
- added ?: , MX, F.Cu at (318.3, 44.4)
- added ?: , MX, F.Cu at (28.4, 63.2)
- added ?: , MX, F.Cu at (47.2, 66.5)
- added ?: , MX, F.Cu at (66.5, 66.8)
- added ?: , MX, F.Cu at (86.1, 65.2)
- added ?: , MX, F.Cu at (103.8, 74.4)
- added ?: , MX, F.Cu at (121.7, 82.7)
- added ?: , MX, F.Cu at (155.9, 106.0)
- added ?: , MX, F.Cu at (175.0, 106.0)
- added ?: , MX, F.Cu at (194.1, 106.0)
- added ?: , MX, F.Cu at (92.7, 27.7)
- added ?: , MX, F.Cu at (228.3, 82.7)
- added ?: , MX, F.Cu at (246.2, 74.4)
- added ?: , MX, F.Cu at (263.9, 65.2)
- added ?: , MX, F.Cu at (283.5, 66.8)
- added ?: , MX, F.Cu at (302.8, 66.5)
- added ?: , MX, F.Cu at (321.6, 63.2)
- added ?: , MX, F.Cu at (25.1, 81.9)
- added ?: , MX, F.Cu at (43.9, 85.2)
- added ?: , MX, F.Cu at (63.2, 85.6)
- added ?: , MX, F.Cu at (82.8, 84.0)
- added ?: , MX, F.Cu at (110.4, 36.9)
- added ?: , MX, F.Cu at (100.5, 93.2)
- added ?: , MX, F.Cu at (118.4, 101.4)
- added ?: , MX, F.Cu at (155.9, 144.1)
- added ?: , MX, F.Cu at (175.0, 125.0)
- added ?: , MX, F.Cu at (194.1, 144.1)
- added ?: , MX, F.Cu at (231.6, 101.4)
- added ?: , MX, F.Cu at (249.5, 93.2)
- added ?: , MX, F.Cu at (267.2, 84.0)
- added ?: , MX, F.Cu at (286.8, 85.6)
- added ?: , MX, F.Cu at (306.1, 85.2)
- added ?: , MX, F.Cu at (128.3, 45.1)
- added ?: , MX, F.Cu at (324.9, 81.9)
- added ?: , MX, F.Cu at (21.8, 100.7)
- added ?: , MX, F.Cu at (40.6, 104.0)
- added ?: , MX, F.Cu at (59.9, 104.3)
- added ?: , MX, F.Cu at (79.5, 102.7)
- added ?: , MX, F.Cu at (97.2, 111.9)
- added ?: , MX, F.Cu at (115.1, 120.2)
- added ?: , MX, F.Cu at (130.6, 142.2)
- added ?: , MX, F.Cu at (175.0, 144.1)
- added ?: , MX, F.Cu at (219.4, 142.2)
- added ?: , MX, F.Cu at (155.9, 67.9)
- added ?: , MX, F.Cu at (234.9, 120.2)
- added ?: , MX, F.Cu at (252.8, 111.9)
- added ?: , MX, F.Cu at (270.5, 102.7)
- added ?: , MX, F.Cu at (290.1, 104.3)
- added ?: , MX, F.Cu at (309.4, 104.0)
- added ?: , MX, F.Cu at (328.2, 100.7)
- added ?: , MX, F.Cu at (18.5, 119.4)
- added ?: , MX, F.Cu at (37.3, 122.7)
- added ?: , MX, F.Cu at (56.6, 123.1)
- added ?: , MX, F.Cu at (76.2, 121.5)
- added ?: , MX, F.Cu at (175.0, 67.9)
- added ?: , MX, F.Cu at (93.9, 130.7)
- added ?: , MX, F.Cu at (111.8, 138.9)
- added ?: , MX, F.Cu at (238.2, 138.9)
- added ?: , MX, F.Cu at (256.1, 130.7)
- added ?: , MX, F.Cu at (273.8, 121.5)
- added ?: , MX, F.Cu at (293.4, 123.1)
- added ?: , MX, F.Cu at (312.7, 122.7)
- added ?: , MX, F.Cu at (331.5, 119.4)
- added ?: , MX, F.Cu at (194.1, 67.9)
- U1: value ItsyBitsy -> Elite-C; footprint ItsyBitsy -> Elite-C; moved to B.Cu
- moved RGB10 79.8 mm to (110.9, 46.4), turned to 260 degrees
- moved RGB1 79.8 mm to (239.1, 46.4), turned to 280 degrees
- moved RGB2 77.9 mm to (278.0, 47.7), turned to 280 degrees
- moved RGB9 77.9 mm to (72.0, 47.7), turned to 260 degrees
- moved RGB11 53.4 mm to (146.5, 63.9), turned to 260 degrees
- moved RGB0 53.4 mm to (203.5, 63.9), turned to 280 degrees
- moved RGB4 36.4 mm to (249.0, 102.7)
- moved RGB7 36.4 mm to (101.0, 102.7)
- moved RGB5 30.4 mm to (213.4, 120.2), turned to 100 degrees
- moved RGB6 30.4 mm to (136.6, 120.2), turned to 80 degrees
- moved U1 29.4 mm to (175.0, 65.0)
- moved RGB3 26.7 mm to (287.9, 104.0)
- moved RGB8 26.7 mm to (62.1, 104.0)
Connections:
- RGB0 pad 1: N-GND-1 -> (no net)
- RGB0 pad 2: N-RGB-D0 -> (no net)
- RGB0 pad 3: N-5V-0 -> (no net)
- RGB0 pad 4: N-RGB-D1 -> (no net)
- RGB1 pad 1: N-GND-1 -> (no net)
- RGB1 pad 2: N-RGB-D1 -> (no net)
- RGB1 pad 3: N-5V-0 -> (no net)
- RGB1 pad 4: N-RGB-D2 -> (no net)
- RGB10 pad 1: N-GND-1 -> (no net)
- RGB10 pad 2: N-RGB-D10 -> (no net)
- RGB10 pad 3: N-5V-0 -> (no net)
- RGB10 pad 4: N-RGB-D11 -> (no net)
- RGB11 pad 1: N-GND-1 -> (no net)
- RGB11 pad 2: N-RGB-D11 -> (no net)
- RGB11 pad 3: N-5V-0 -> (no net)
- RGB2 pad 1: N-GND-1 -> (no net)
- RGB2 pad 2: N-RGB-D2 -> (no net)
- RGB2 pad 3: N-5V-0 -> (no net)
- RGB2 pad 4: N-RGB-D3 -> (no net)
- RGB3 pad 1: N-GND-1 -> (no net)
- RGB3 pad 2: N-RGB-D3 -> (no net)
- RGB3 pad 3: N-5V-0 -> (no net)
- RGB3 pad 4: N-RGB-D4 -> (no net)
- RGB4 pad 1: N-GND-1 -> (no net)
- RGB4 pad 2: N-RGB-D4 -> (no net)
- RGB4 pad 3: N-5V-0 -> (no net)
- RGB4 pad 4: N-RGB-D5 -> (no net)
- RGB5 pad 1: N-GND-1 -> (no net)
- RGB5 pad 2: N-RGB-D5 -> (no net)
- RGB5 pad 3: N-5V-0 -> (no net)
- RGB5 pad 4: N-RGB-D6 -> (no net)
- RGB6 pad 1: N-GND-1 -> (no net)
- RGB6 pad 2: N-RGB-D6 -> (no net)
- RGB6 pad 3: N-5V-0 -> (no net)
- RGB6 pad 4: N-RGB-D7 -> (no net)
- RGB7 pad 1: N-GND-1 -> (no net)
- RGB7 pad 2: N-RGB-D7 -> (no net)
- RGB7 pad 3: N-5V-0 -> (no net)
- RGB7 pad 4: N-RGB-D8 -> (no net)
- RGB8 pad 1: N-GND-1 -> (no net)
- RGB8 pad 2: N-RGB-D8 -> (no net)
- RGB8 pad 3: N-5V-0 -> (no net)
- RGB8 pad 4: N-RGB-D9 -> (no net)
- RGB9 pad 1: N-GND-1 -> (no net)
- RGB9 pad 2: N-RGB-D9 -> (no net)
- RGB9 pad 3: N-5V-0 -> (no net)
- RGB9 pad 4: N-RGB-D10 -> (no net)
- U1 pad 1: N-RST -> (no net)
- U1 pad 10: N-col-5 -> (no net)
- U1 pad 11: N-col-6 -> (no net)
- U1 pad 12: N-row-5 -> (no net)
- U1 pad 17: N-col-7 -> (no net)
- U1 pad 18: N-RGB-D0 -> (no net)
- U1 pad 19: N-row-4 -> (no net)
- U1 pad 2: N-5V-0 -> (no net)
- U1 pad 20: N-row-3 -> (no net)
- U1 pad 21: N-row-2 -> (no net)
- U1 pad 22: N-row-1 -> (no net)
- U1 pad 23: N-row-0 -> (no net)
- U1 pad 24: N-col-8 -> (no net)
- U1 pad 25: N-col-9 -> (no net)
- U1 pad 26: N-col-10 -> (no net)
- U1 pad 27: N-col-11 -> (no net)
- U1 pad 28: N-col-12 -> (no net)
- U1 pad 29: N-col-13 -> (no net)
- U1 pad 4: N-GND-0 -> (no net)
- U1 pad 5: N-col-0 -> (no net)
- U1 pad 6: N-col-1 -> (no net)
- U1 pad 7: N-col-2 -> (no net)
- U1 pad 8: N-col-3 -> (no net)
- U1 pad 9: N-col-4 -> (no net)
Routing:
- net N-GND-1: track 931.7 -> 0.00 mm, vias 14 -> 0
- net N-5V-0: track 888.3 -> 0.00 mm, vias 14 -> 0
- net N-row-5: track 579.2 -> 0.00 mm, vias 1 -> 0
- net N-row-4: track 460.1 -> 0.00 mm, vias 1 -> 0
- net N-row-3: track 417.5 -> 0.00 mm, vias 1 -> 0
- net N-row-2: track 409.9 -> 0.00 mm, vias 1 -> 0
- net N-row-1: track 383.2 -> 0.00 mm, vias 1 -> 0
- net N-row-0: track 380.9 -> 0.00 mm
- net N-col-0: track 243.6 -> 0.00 mm
- net N-col-14: track 235.7 -> 0.00 mm
- net N-col-1: track 230.1 -> 0.00 mm
- net N-col-13: track 224.6 -> 0.00 mm
- net N-col-2: track 216.2 -> 0.00 mm
- net N-col-12: track 207.4 -> 0.00 mm
- net N-col-3: track 193.6 -> 0.00 mm
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Other:
- board size 322.7 x 132.7 mm -> 287.6 x 118.8 mm
- board text removed: "Bloomer"
- board text removed: "By: CozyKeys"
- board text removed: "RST"

Commit message: Progress
Parts:
- removed ? (x87): , MX
- removed RGB0, RGB1, RGB10, RGB11, RGB2, RGB3, RGB4, RGB5, RGB6, RGB7, RGB8, RGB9: VAL**, WS2812B
- added D0:0: , DIODE, F.Cu at (52.9, 27.0)
- added D0:1: , DIODE, F.Cu at (71.7, 30.3)
- added D0:10: , DIODE, F.Cu at (241.7, 38.3)
- added D0:11: , DIODE, F.Cu at (259.4, 29.1)
- added D0:12: , DIODE, F.Cu at (279.0, 30.7)
- added D0:13: , DIODE, F.Cu at (298.3, 30.3)
- added D0:14: , DIODE, F.Cu at (317.1, 27.0)
- added D0:2: , DIODE, F.Cu at (91.0, 30.7)
- added D0:3: , DIODE, F.Cu at (110.6, 29.1)
- added D0:4: , DIODE, F.Cu at (128.3, 38.3)
- added D0:5: , DIODE, F.Cu at (146.2, 46.5)
- added D0:6: , DIODE, F.Cu at (173.9, 48.9)
- added D0:7: , DIODE, F.Cu at (193.0, 48.9)
- added D0:8: , DIODE, F.Cu at (212.1, 48.9)
- added D0:9: , DIODE, F.Cu at (223.8, 46.5)
- added D1:0: , DIODE, F.Cu at (49.6, 45.8)
- added D1:1: , DIODE, F.Cu at (68.4, 49.1)
- added D1:10: , DIODE, F.Cu at (245.0, 57.0)
- added D1:11: , DIODE, F.Cu at (262.7, 47.8)
- added D1:12: , DIODE, F.Cu at (282.3, 49.4)
- added D1:13: , DIODE, F.Cu at (301.6, 49.1)
- added D1:14: , DIODE, F.Cu at (320.4, 45.8)
- added D1:2: , DIODE, F.Cu at (87.7, 49.4)
- added D1:3: , DIODE, F.Cu at (107.3, 47.8)
- added D1:4: , DIODE, F.Cu at (125.0, 57.0)
- added D1:5: , DIODE, F.Cu at (142.9, 65.3)
- added D1:6: , DIODE, F.Cu at (173.9, 77.5)
- added D1:7: , DIODE, F.Cu at (193.0, 77.5)
- added D1:8: , DIODE, F.Cu at (212.1, 77.5)
- added D1:9: , DIODE, F.Cu at (227.1, 65.3)
- added D2:0: , DIODE, F.Cu at (46.3, 64.5)
- added D2:1: , DIODE, F.Cu at (65.1, 67.9)
- added D2:10: , DIODE, F.Cu at (248.3, 75.8)
- added D2:11: , DIODE, F.Cu at (266.0, 66.6)
- added D2:12: , DIODE, F.Cu at (285.6, 68.2)
- added D2:13: , DIODE, F.Cu at (304.9, 67.9)
- added D2:14: , DIODE, F.Cu at (323.7, 64.5)
- added D2:2: , DIODE, F.Cu at (84.4, 68.2)
- added D2:3: , DIODE, F.Cu at (104.0, 66.6)
- added D2:4: , DIODE, F.Cu at (121.7, 75.8)
- added D2:5: , DIODE, F.Cu at (139.6, 84.0)
- added D2:6: , DIODE, F.Cu at (173.9, 96.5)
- added D2:7: , DIODE, F.Cu at (193.0, 96.5)
- added D2:8: , DIODE, F.Cu at (212.1, 96.5)
- added D2:9: , DIODE, F.Cu at (230.4, 84.0)
- added D3:0: , DIODE, F.Cu at (43.0, 83.3)
- added D3:1: , DIODE, F.Cu at (61.8, 86.6)
- added D3:10: , DIODE, F.Cu at (251.6, 94.6)
- added D3:11: , DIODE, F.Cu at (269.3, 85.4)
- added D3:12: , DIODE, F.Cu at (288.9, 87.0)
- added D3:13: , DIODE, F.Cu at (308.2, 86.6)
- added D3:14: , DIODE, F.Cu at (327.0, 83.3)
- added D3:2: , DIODE, F.Cu at (81.1, 87.0)
- added D3:3: , DIODE, F.Cu at (100.7, 85.4)
- added D3:4: , DIODE, F.Cu at (118.4, 94.6)
- added D3:5: , DIODE, F.Cu at (136.3, 102.8)
- added D3:6: , DIODE, F.Cu at (173.9, 144.1)
- added D3:7: , DIODE, F.Cu at (193.0, 125.1)
- added D3:8: , DIODE, F.Cu at (212.1, 144.1)
- added D3:9: , DIODE, F.Cu at (233.7, 102.8)
- added D4:0: , DIODE, F.Cu at (39.7, 102.1)
- added D4:1: , DIODE, F.Cu at (58.5, 105.4)
- added D4:10: , DIODE, F.Cu at (254.9, 113.3)
- added D4:11: , DIODE, F.Cu at (272.6, 104.1)
- added D4:12: , DIODE, F.Cu at (292.3, 105.7)
- added D4:13: , DIODE, F.Cu at (311.5, 105.4)
- added D4:14: , DIODE, F.Cu at (330.3, 102.1)
- added D4:2: , DIODE, F.Cu at (77.7, 105.7)
- added D4:3: , DIODE, F.Cu at (97.4, 104.1)
- added D4:4: , DIODE, F.Cu at (115.1, 113.3)
- added D4:5: , DIODE, F.Cu at (133.0, 121.6)
- added D4:6: , DIODE, F.Cu at (148.4, 143.6)
- added D4:7: , DIODE, F.Cu at (193.0, 144.1)
- added D4:8: , DIODE, F.Cu at (237.3, 140.9)
- added D4:9: , DIODE, F.Cu at (237.0, 121.6)
- added D5:0: , DIODE, F.Cu at (36.4, 120.8)
- added D5:1: , DIODE, F.Cu at (55.2, 124.1)
- added D5:10: , DIODE, F.Cu at (258.2, 132.1)
- added D5:11: , DIODE, F.Cu at (275.9, 122.9)
- added D5:12: , DIODE, F.Cu at (295.6, 124.5)
- added D5:13: , DIODE, F.Cu at (314.8, 124.1)
- added D5:14: , DIODE, F.Cu at (333.6, 120.8)
- added D5:2: , DIODE, F.Cu at (74.4, 124.5)
- added D5:3: , DIODE, F.Cu at (94.1, 122.9)
- added D5:4: , DIODE, F.Cu at (111.8, 132.1)
- added D5:5: , DIODE, F.Cu at (129.7, 140.3)
- added D5:9: , DIODE, F.Cu at (240.3, 140.3)
- added SW0:0: , MX, F.Cu at (45.1, 25.6)
- added SW0:1: , MX, F.Cu at (63.8, 28.9)
- added SW0:10: , MX, F.Cu at (249.6, 36.9)
- added SW0:11: , MX, F.Cu at (267.3, 27.7)
- added SW0:12: , MX, F.Cu at (286.9, 29.3)
- added SW0:13: , MX, F.Cu at (306.2, 28.9)
- added SW0:14: , MX, F.Cu at (324.9, 25.6)
- added SW0:2: , MX, F.Cu at (83.1, 29.3)
- added SW0:3: , MX, F.Cu at (102.7, 27.7)
- added SW0:4: , MX, F.Cu at (120.4, 36.9)
- added SW0:5: , MX, F.Cu at (138.3, 45.1)
- added SW0:6: , MX, F.Cu at (165.9, 48.9)
- added SW0:7: , MX, F.Cu at (185.0, 48.9)
- added SW0:8: , MX, F.Cu at (204.1, 48.9)
- added SW0:9: , MX, F.Cu at (231.7, 45.1)
- added SW1:0: , MX, F.Cu at (41.7, 44.4)
- added SW1:1: , MX, F.Cu at (60.5, 47.7)
- added SW1:10: , MX, F.Cu at (252.9, 55.7)
- added SW1:11: , MX, F.Cu at (270.6, 46.4)
- added SW1:12: , MX, F.Cu at (290.2, 48.1)
- added SW1:13: , MX, F.Cu at (309.5, 47.7)
- added SW1:14: , MX, F.Cu at (328.3, 44.4)
- added SW1:2: , MX, F.Cu at (79.8, 48.1)
- added SW1:3: , MX, F.Cu at (99.4, 46.4)
- added SW1:4: , MX, F.Cu at (117.1, 55.7)
- added SW1:5: , MX, F.Cu at (135.0, 63.9)
- added SW1:6: , MX, F.Cu at (165.9, 77.5)
- added SW1:7: , MX, F.Cu at (185.0, 77.5)
- added SW1:8: , MX, F.Cu at (204.1, 77.5)
- added SW1:9: , MX, F.Cu at (235.0, 63.9)
- added SW2:0: , MX, F.Cu at (38.4, 63.2)
- added SW2:1: , MX, F.Cu at (57.2, 66.5)
- added SW2:10: , MX, F.Cu at (256.2, 74.4)
- added SW2:11: , MX, F.Cu at (273.9, 65.2)
- added SW2:12: , MX, F.Cu at (293.5, 66.8)
- added SW2:13: , MX, F.Cu at (312.8, 66.5)
- added SW2:14: , MX, F.Cu at (331.6, 63.2)
- added SW2:2: , MX, F.Cu at (76.5, 66.8)
- added SW2:3: , MX, F.Cu at (96.1, 65.2)
- added SW2:4: , MX, F.Cu at (113.8, 74.4)
- added SW2:5: , MX, F.Cu at (131.7, 82.7)
- added SW2:6: , MX, F.Cu at (165.9, 96.5)
- added SW2:7: , MX, F.Cu at (185.0, 96.5)
- added SW2:8: , MX, F.Cu at (204.1, 96.5)
- added SW2:9: , MX, F.Cu at (238.3, 82.7)
- added SW3:0: , MX, F.Cu at (35.1, 81.9)
- added SW3:1: , MX, F.Cu at (53.9, 85.2)
- added SW3:10: , MX, F.Cu at (259.5, 93.2)
- added SW3:11: , MX, F.Cu at (277.2, 84.0)
- added SW3:12: , MX, F.Cu at (296.8, 85.6)
- added SW3:13: , MX, F.Cu at (316.1, 85.2)
- added SW3:14: , MX, F.Cu at (334.9, 81.9)
- added SW3:2: , MX, F.Cu at (73.2, 85.6)
- added SW3:3: , MX, F.Cu at (92.8, 84.0)
- added SW3:4: , MX, F.Cu at (110.5, 93.2)
- added SW3:5: , MX, F.Cu at (128.4, 101.4)
- added SW3:6: , MX, F.Cu at (165.9, 144.1)
- added SW3:7: , MX, F.Cu at (185.0, 125.1)
- added SW3:8: , MX, F.Cu at (204.1, 144.1)
- added SW3:9: , MX, F.Cu at (241.6, 101.4)
- added SW4:0: , MX, F.Cu at (31.8, 100.7)
- added SW4:1: , MX, F.Cu at (50.6, 104.0)
- added SW4:10: , MX, F.Cu at (262.8, 111.9)
- added SW4:11: , MX, F.Cu at (280.5, 102.7)
- added SW4:12: , MX, F.Cu at (300.1, 104.3)
- added SW4:13: , MX, F.Cu at (319.4, 104.0)
- added SW4:14: , MX, F.Cu at (338.2, 100.7)
- added SW4:2: , MX, F.Cu at (69.9, 104.3)
- added SW4:3: , MX, F.Cu at (89.5, 102.7)
- added SW4:4: , MX, F.Cu at (107.2, 111.9)
- added SW4:5: , MX, F.Cu at (125.1, 120.2)
- added SW4:6: , MX, F.Cu at (140.6, 142.2)
- added SW4:7: , MX, F.Cu at (185.0, 144.1)
- added SW4:8: , MX, F.Cu at (229.4, 142.2)
- added SW4:9: , MX, F.Cu at (244.9, 120.2)
- added SW5:0: , MX, F.Cu at (28.5, 119.4)
- added SW5:1: , MX, F.Cu at (47.3, 122.7)
- added SW5:10: , MX, F.Cu at (266.1, 130.7)
- added SW5:11: , MX, F.Cu at (283.8, 121.5)
- added SW5:12: , MX, F.Cu at (303.4, 123.1)
- added SW5:13: , MX, F.Cu at (322.7, 122.7)
- added SW5:14: , MX, F.Cu at (341.5, 119.4)
- added SW5:2: , MX, F.Cu at (66.6, 123.1)
- added SW5:3: , MX, F.Cu at (86.2, 121.5)
- added SW5:4: , MX, F.Cu at (103.9, 130.7)
- added SW5:5: , MX, F.Cu at (121.8, 138.9)
- added SW5:9: , MX, F.Cu at (248.2, 138.9)
- moved U1 13.7 mm to (185.0, 55.6)
Other:
- board size 287.6 x 118.8 mm -> 333.9 x 138 mm
