File: pcb/bloomer_v4.sch (KiCad schematic (older format))
At the start: 183 parts, among them K01 MX, K02 MX, K03 MX, K04 MX, K05 MX, K06 MX, K07 MX, K08 MX, K09 MX, K10 MX, K11 MX, K12 MX, K13 MX, K14 MX, K15 MX, K16 MX, K17 MX, K18 MX, K19 MX, K20 MX, K21 MX, K22 MX, K23 MX, K24 MX, K25 MX, K26 MX, K27 MX, K28 MX, K29 MX, K30 MX, K31 MX, K32 MX, K33 MX, K34 MX, K35 MX, K36 MX, K37 MX, K38 MX, K39 MX, K40 MX, K41 MX, K42 MX, K43 MX, K44 MX, K45 MX, K46 MX, K47 MX, K48 MX, K49 MX, K50 MX, K51 MX, K52 MX, K53 MX, K54 MX, K55 MX, K56 MX, K57 MX, K58 MX, K59 MX, K60 MX, K61 MX, K62 MX, K63 MX, K64 MX, K65 MX, K66 MX, K67 MX, K68 MX, K69 MX, K70 MX, K71 MX, K72 MX, K73 MX, K74 MX, K75 MX, K76 MX, K77 MX, K78 MX, K79 MX, K80 MX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

Commit message: Updates
Parts:
- added C10, C11, C12, C13, C14, C15, C16, C17, C18, C19, C20, C9: 100n, Capacitor_SMD:C_0805_2012Metric_Pad1.18x1.45mm_HandSolder, symbol Device:C_Small
- added C8: 1u, Capacitor_SMD:C_0805_2012Metric_Pad1.18x1.45mm_HandSolder, symbol Device:C_Small
- added J1, J2: Conn_01x04, cozy-parts:MX_1.00u, symbol Connector_Generic:Conn_01x04
- added J3: USB_C_Receptacle, cozy-parts:MX_1.00u, symbol Connector:USB_C_Receptacle
- added L1, L10, L11, L12, L2, L3, L4, L5, L6, L7, L8, L9: WS2812B, LED_SMD:LED_WS2812B_PLCC4_5.0x5.0mm_P3.2mm, symbol LED:WS2812B
- added R1, R2: 10k, Resistor_SMD:R_0805_2012Metric_Pad1.20x1.40mm_HandSolder, symbol Device:R
- added R3, R4: 22, Resistor_SMD:R_0805_2012Metric_Pad1.20x1.40mm_HandSolder, symbol Device:R
- added R5, R6: 5.1k, Resistor_SMD:R_0805_2012Metric_Pad1.20x1.40mm_HandSolder, symbol Device:R
- added SW1: SW_Push, cozy-parts:SW_TH_Tactile_Omron_B3F-10xx, symbol Switch:SW_Push
- C1, C2, C3, C4, C5, C6, C7: footprint (none) -> Capacitor_SMD:C_0805_2012Metric_Pad1.18x1.45mm_HandSolder
- D01, D02, D03, D04, D05, D06, D07, D08, D09, D10, D11, D12, D13, D14, D15, D16, D17, D18, D19, D20, D21, D22, D23, D24, D25, D26, D27, D28, D29, D30, D31, D32, D33, D34, D35, D36, D37, D38, D39, D40, D41, D42, D43, D44, D45, D46, D47, D48, D49, D50, D51, D52, D53, D54, D55, D56, D57, D58, D59, D60, D61, D62, D63, D64, D65, D66, D67, D68, D69, D70, D71, D72, D73, D74, D75, D76, D77, D78, D79, D80, D81, D82, D83, D84, D85, D86: footprint (none) -> Diode_SMD:D_SOD-123F
- D87, K01, K02, K03, K04, K05, K06, K07, K08, K09, K10, K11, K12, K13, K14, K15, K16, K17, K18, K19, K20, K21, K22, K23, K24, K25, K26, K27, K28, K29, K30, K31, K32, K33, K34, K35, K36, K37, K38, K39, K40, K41, K42, K43, K44, K45, K46, K47, K48, K49, K50, K51, K52, K53, K54, K55, K56, K57, K58, K59, K60, K61, K62, K63, K64, K65, K66, K67, K68, K69, K70, K71, K72, K73, K74, K75, K76, K77, K78, K79, K80, K81, K82, K83, K84, K85, K86, K87: footprint (none) -> cozy-parts:MX_1.00u
- U1: renamed from U?; footprint (none) -> Keebio-Parts:ATMEGA32U4-AU
- Y1: footprint (none) -> Crystal:Crystal_SMD_SeikoEpson_FA238-4Pin_3.2x2.5mm_HandSoldering
Connections:
- net GND: now also U1.15 (GND), U1.23 (GND), U1.35 (GND), U1.43 (GND), U1.5 (UGnd), C10.1, C11.1, C12.1, C13.1, C14.1, C15.1, C16.1, C17.1, C18.1, C19.1, C20.1, C8.2, C9.1, J1.1 (Pin_1), J3.A1 (GND), J3.A12 (GND), J3.B1 (GND), J3.B12 (GND), J3.S1 (SHIELD), L1.3 (VSS), L10.3 (VSS), L11.3 (VSS), L12.3 (VSS), L2.3 (VSS), L3.3 (VSS), L4.3 (VSS), L5.3 (VSS), L6.3 (VSS), L7.3 (VSS), L8.3 (VSS), L9.3 (VSS), R2.1, R5.1, R6.1, SW1.1
- net VCC: now also U1.14 (VCC), U1.2 (UVcc), U1.24 (AVCC), U1.34 (VCC), U1.44 (AVCC), U1.7 (VBus), C10.2, C11.2, C12.2, C13.2, C14.2, C15.2, C16.2, C17.2, C18.2, C19.2, C20.2, C9.2, J1.2 (Pin_2), J3.A4 (VBUS), J3.A9 (VBUS), J3.B4 (VBUS), J3.B9 (VBUS), L1.1 (VDD), L10.1 (VDD), L11.1 (VDD), L12.1 (VDD), L2.1 (VDD), L3.1 (VDD), L4.1 (VDD), L5.1 (VDD), L6.1 (VDD), L7.1 (VDD), L8.1 (VDD), L9.1 (VDD), R1.2
- net col0: now also U1.8 (PB0/SS)
- net col1: now also U1.9 (PB1/SCK)
- net col10: now also U1.26 (T1/PD6)
- net col11: now also U1.27 (T0/PD7)
- net col12: now also U1.28 (PB4)
- net col13: now also U1.29 (PB5)
- net col14: now also U1.30 (PB6)
- net col2: now also U1.10 (PB2/MOSI)
- net col3: now also U1.11 (PB3/MISO)
- net col4: now also U1.12 (PB7/~RTS)
- net col5: now also U1.1 (PE6/AIN0)
- net col6: now also U1.20 (PD2/RXD1)
- net col7: now also U1.21 (PD3/TXD1)
- net col8: now also U1.22 (PD5/XCK1)
- net col9: now also U1.25 (ICP1/PD4)
- net row0: now also U1.41 (PF0)
- net row1: now also U1.40 (PF1)
- net row2: now also U1.39 (PF4)
- net row3: now also U1.38 (PF5)
- net row4: now also U1.37 (PF6)
- net row5: now also U1.36 (PF7)
- net at U1.13 (~RESET): now also R1.1, SW1.2
- net scl: now reaches U1.18 (PD0/INT0)
- net scl: now also J1.3 (Pin_3)
- net sda: now reaches U1.19 (PD1/INT1)
- net sda: now also J1.4 (Pin_4)
- net usb_d-: now reaches U1.3 (D-)
- net usb_d-: now also R3.1
- net rgb: now reaches U1.31 (PC6)
- net rgb: now also L1.4 (DIN)
- net at U1.33 (~HWB/PE2): now also R2.2
- net usb_d+: now reaches U1.4 (D+)
- net usb_d+: now also R4.1
- net usb_cap: now reaches U1.6 (UCap)
- net usb_cap: now also C8.1
- new net: L1.2 (DOUT), L2.4 (DIN)
- new net: L2.2 (DOUT), L3.4 (DIN)
- new net: L3.2 (DOUT), L4.4 (DIN)
- new net: L4.2 (DOUT), L5.4 (DIN)
- new net: L5.2 (DOUT), L6.4 (DIN)
- new net: L6.2 (DOUT), L7.4 (DIN)
- new net: L11.2 (DOUT), L12.4 (DIN)
- new net: L10.2 (DOUT), L11.4 (DIN)
- new net: L10.4 (DIN), L9.2 (DOUT)
- new net: L8.2 (DOUT), L9.4 (DIN)
- new net: L7.2 (DOUT), L8.4 (DIN)
- new net: J3.A5 (CC1), R5.2
- new net: J3.A6 (D+), J3.B6 (D+), R4.2
- new net: J3.A7 (D-), J3.B7 (D-), R3.2
- new net: J3.B5 (CC2), R6.2
- no-connect marks 0 -> 16
Other:
- moved on the sheet: C1, C2, C3, C4, C5, C6, C7, U1, Y1
