File: pcb/bloomer_v4.sch (KiCad schematic (older format))
At the start: 217 parts, among them K00 MX, K01 MX, K02 MX, K03 MX, K04 MX, K05 MX, K06 MX, K07 MX, K08 MX, K09 MX, K10 MX, K11 MX, K12 MX, K13 MX, K14 MX, K15 MX, K16 MX, K17 MX, K18 MX, K19 MX, K20 MX, K21 MX, K22 MX, K23 MX, K24 MX, K25 MX, K26 MX, K27 MX, K28 MX, K29 MX, K30 MX, K31 MX, K32 MX, K33 MX, K34 MX, K35 MX, K36 MX, K37 MX, K38 MX, K39 MX, K40 MX, K41 MX, K42 MX, K43 MX, K44 MX, K45 MX, K46 MX, K47 MX, K48 MX, K49 MX, K50 MX, K51 MX, K52 MX, K53 MX, K54 MX, K55 MX, K56 MX, K57 MX, K58 MX, K59 MX, K60 MX, K61 MX, K62 MX, K63 MX, K64 MX, K65 MX, K66 MX, K67 MX, K68 MX, K69 MX, K70 MX, K71 MX, K72 MX, K73 MX, K74 MX, K75 MX, K76 MX, K77 MX, K78 MX, K79 MX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

Commit message: Updates
Parts:
- removed OLED1: Conn_01x04, cozy-parts:hiletgo_128x32_oled, symbol Connector_Generic:Conn_01x04
Connections:
- net scl: no longer names the net of MCU1.18 (PD0/INT0)
- net sda: no longer names the net of MCU1.19 (PD1/INT1)
- no-connect marks 5 -> 7
Changed lines of the file:
@@
 	0    1    1    0
 $EndComp
-Text Label 2350 6750 2    50   ~ 0
-scl
-Text Label 2350 6850 2    50   ~ 0
-sda
 Text Label 2350 5050 2    50   ~ 0
 col5
@@
 	1200 4700 1050 4700
 Connection ~ 1200 4700
-$Comp
-L Connector_Generic:Conn_01x04 OLED1
-U 1 1 62126141
-P 7300 5400
-F 0 "OLED1" H 7218 5717 50  0000 C CNN
-F 1 "Conn_01x04" H 7218 5626 50  0000 C CNN
-F 2 "cozy-parts:hiletgo_128x32_oled" H 7300 5400 50  0001 C CNN
-F 3 "~" H 7300 5400 50  0001 C CNN
-	1    7300 5400
-	-1   0    0    -1
-$EndComp
-$Comp
-L power:GND #PWR0137
-U 1 1 6214F827
-P 7500 5300
-F 0 "#PWR0137" H 7500 5050 50  0001 C CNN
-F 1 "GND" V 7505 5172 50  0000 R CNN
-F 2 "" H 7500 5300 50  0001 C CNN
-F 3 "" H 7500 5300 50  0001 C CNN
-	1    7500 5300
-	0    -1   -1   0
-$EndComp
-$Comp
-L power:VCC #PWR0138
-U 1 1 62150385
-P 7500 5400
-F 0 "#PWR0138" H 7500 5250 50  0001 C CNN
-F 1 "VCC" V 7515 5528 50  0000 L CNN
-F 2 "" H 7500 5400 50  0001 C CNN
-F 3 "" H 7500 5400 50  0001 C CNN
-	1    7500 5400
-	0    1    1    0
-$EndComp
-Text Label 7500 5500 0    50   ~ 0
-scl
-Text Label 7500 5600 0    50   ~ 0
-sda
+NoConn ~ 2350 6850
+NoConn ~ 2350 6750
 $EndSCHEMATC
