File: pcb/bloomer_v4.kicad_pcb (KiCad board)
At the start: 2 copper layers, 218 parts, among them J1 Conn_01x04, J2 Conn_01x04, J3 USB_C_Receptacle, K01 MX, K02 MX, K03 MX, K04 MX, K05 MX, K06 MX, K07 MX, K08 MX, K09 MX, K10 MX, K11 MX, K12 MX, K13 MX, K14 MX, K15 MX, K16 MX, K17 MX, K18 MX, K19 MX, K20 MX, K21 MX, K22 MX, K23 MX, K24 MX, K25 MX, K26 MX, K27 MX, K28 MX, K29 MX, K30 MX, K31 MX, K32 MX, K33 MX, K34 MX, K35 MX, K36 MX, K37 MX, K38 MX, K39 MX, K40 MX, K41 MX, K42 MX, K43 MX, K44 MX, K45 MX, K46 MX, K47 MX, K48 MX, K49 MX, K50 MX, K51 MX, K52 MX, K53 MX, K54 MX, K55 MX, K56 MX, K57 MX, K58 MX, K59 MX, K60 MX, K61 MX, K62 MX, K63 MX, K64 MX, K65 MX, K66 MX, K67 MX, K68 MX, K69 MX, K70 MX, K71 MX, K72 MX, K73 MX, K74 MX, K75 MX, K76 MX, K77 MX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

Commit message: Updates
Parts:
- removed D87: D_Small, cozy-parts:MX_1.00u
- removed J1, J2: Conn_01x04, cozy-parts:MX_1.00u
- removed J3: USB_C_Receptacle, cozy-parts:MX_1.00u
- removed K87: MX, cozy-parts:MX_1.00u
- removed L1, L10, L11, L12, L2, L3, L4, L5, L6, L7, L8, L9: WS2812B, LED_SMD:LED_WS2812B_PLCC4_5.0x5.0mm_P3.2mm
- removed U1: ATMEGA32U4, Keebio-Parts:ATMEGA32U4-AU
- added D00: D_Small, Keebio-Parts:Diode-dual, B.Cu at (66.4, 42.3)
- added K00: MX, cozy-parts:MX_1.00u, F.Cu at (58.2, 40.8)
- added LED1: WS2812B, LED_SMD:LED_WS2812B_PLCC4_5.0x5.0mm_P3.2mm, B.Cu at (250.1, 69.7)
- added LED10: WS2812B, LED_SMD:LED_WS2812B_PLCC4_5.0x5.0mm_P3.2mm, B.Cu at (75.3, 53.5)
- added LED11: WS2812B, LED_SMD:LED_WS2812B_PLCC4_5.0x5.0mm_P3.2mm, B.Cu at (114.2, 52.2)
- added LED12: WS2812B, LED_SMD:LED_WS2812B_PLCC4_5.0x5.0mm_P3.2mm, B.Cu at (149.9, 69.7)
- added LED2: WS2812B, LED_SMD:LED_WS2812B_PLCC4_5.0x5.0mm_P3.2mm, B.Cu at (285.8, 52.2)
- added LED3: WS2812B, LED_SMD:LED_WS2812B_PLCC4_5.0x5.0mm_P3.2mm, B.Cu at (324.7, 53.5)
- added LED4: WS2812B, LED_SMD:LED_WS2812B_PLCC4_5.0x5.0mm_P3.2mm, B.Cu at (337.9, 128.6)
- added LED5: WS2812B, LED_SMD:LED_WS2812B_PLCC4_5.0x5.0mm_P3.2mm, B.Cu at (299.0, 127.3)
- added LED6: WS2812B, LED_SMD:LED_WS2812B_PLCC4_5.0x5.0mm_P3.2mm, B.Cu at (263.4, 144.7)
- added LED7: WS2812B, LED_SMD:LED_WS2812B_PLCC4_5.0x5.0mm_P3.2mm, B.Cu at (136.6, 144.7)
- added LED8: WS2812B, LED_SMD:LED_WS2812B_PLCC4_5.0x5.0mm_P3.2mm, B.Cu at (101.0, 127.3)
- added LED9: WS2812B, LED_SMD:LED_WS2812B_PLCC4_5.0x5.0mm_P3.2mm, B.Cu at (62.1, 128.6)
- added MCU1: ATMEGA32U4, Keebio-Parts:ATMEGA32U4-AU, B.Cu at (168.9, 135.9)
- added OLED1: Conn_01x04, cozy-parts:hiletgo_128x32_oled, B.Cu at (200.0, 47.0)
- added USB1: HRO-TYPE-C-31-M-12, Keebio-Parts:HRO-TYPE-C-31-M-12-Assembly, B.Cu at (200.0, 36.0)
- C1, C10, C11, C12, C13, C14, C15, C16, C17, C18, C19, C2, C20, C3, C4, C5, C6, C7, C8, C9, R1, R2, R3, R4, R5, R6, Y1: moved to B.Cu
- D01, D02, D03, D04, D05, D06, D07, D08, D09, D10, D11, D12, D13, D14, D15, D16, D17, D18, D19, D20, D21, D22, D23, D24, D25, D26, D27, D28, D29, D30, D31, D32, D33, D34, D35, D36, D37, D38, D39, D40, D41, D42, D43, D44, D45, D46, D47, D48, D49, D50, D51, D52, D53, D54, D55, D56, D57, D58, D59, D60, D61, D62, D63, D64, D65, D66, D67, D68, D69, D70, D71, D72, D73, D74, D75, D76, D77, D78, D79, D80, D81, D82, D83, D84, D85, D86: footprint Diode_SMD:D_SOD-123F -> Keebio-Parts:Diode-dual; moved to B.Cu
- SW1: footprint cozy-parts:SW_TH_Tactile_Omron_B3F-10xx -> cozy-parts:SW_TH_Tactile_Omron_B3F-10xx_Centered; moved to B.Cu
- moved K86 329.3 mm to (358.3, 134.6), turned to 10 degrees
- moved K84 309.9 mm to (320.3, 138.3), turned to 10 degrees
- moved K85 293.3 mm to (339.6, 137.9), turned to 10 degrees
- moved K44 274.1 mm to (348.4, 78.3), turned to 10 degrees
- moved K26 266.7 mm to (287.4, 61.6), turned to 10 degrees
- moved C17 265.4 mm to (55.9, 129.1), turned to 350 degrees
- moved K57 261.5 mm to (351.7, 97.1), turned to 10 degrees
- moved D72 261.5 mm to (346.9, 117.3), turned to 280 degrees
- moved K81 243.6 mm to (265.0, 154.1), turned to 10 degrees
- moved D71 237.2 mm to (328.1, 120.6), turned to 280 degrees
- moved D84 233.3 mm to (312.1, 139.7), turned to 280 degrees
- moved K43 229.7 mm to (329.6, 81.7), turned to 10 degrees
- moved C18 229.0 mm to (81.5, 53.0), turned to 170 degrees
- moved D68 228.1 mm to (271.5, 128.6), turned to 280 degrees
- moved K83 227.3 mm to (300.6, 136.7), turned to 10 degrees
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Connections:
- C8 pad 1: /usb_cap -> GND
- C8 pad 2: GND -> /usb_cap
- D15 pad 1: /row0 -> /row1
- D30 pad 1: /row1 -> /row2
- D45 pad 1: /row2 -> /row3
- D58 pad 1: /row3 -> /row4
- D73 pad 1: /row4 -> /row5
- K01 pad 2: /col0 -> /col1
- K02 pad 2: /col1 -> /col2
- K03 pad 2: /col2 -> /col3
- K04 pad 2: /col3 -> /col4
- K05 pad 2: /col4 -> /col5
- K06 pad 2: /col5 -> /col6
- K07 pad 2: /col6 -> /col7
- K08 pad 2: /col7 -> /col8
- K09 pad 2: /col8 -> /col9
- K10 pad 2: /col9 -> /col10
- K11 pad 2: /col10 -> /col11
- K12 pad 2: /col11 -> /col12
- K13 pad 2: /col12 -> /col13
- K14 pad 2: /col13 -> /col14
- K15 pad 2: /col14 -> /col0
- K16 pad 2: /col0 -> /col1
- K17 pad 2: /col1 -> /col2
- K18 pad 2: /col2 -> /col3
- K19 pad 2: /col3 -> /col4
- K20 pad 2: /col4 -> /col5
- K21 pad 2: /col5 -> /col6
- K22 pad 2: /col6 -> /col7
- K23 pad 2: /col7 -> /col8
- K24 pad 2: /col8 -> /col9
- K25 pad 2: /col9 -> /col10
- K26 pad 2: /col10 -> /col11
- K27 pad 2: /col11 -> /col12
- K28 pad 2: /col12 -> /col13
- K29 pad 2: /col13 -> /col14
- K30 pad 2: /col14 -> /col0
- K31 pad 2: /col0 -> /col1
- K32 pad 2: /col1 -> /col2
- K33 pad 2: /col2 -> /col3
- K34 pad 2: /col3 -> /col4
- K35 pad 2: /col4 -> /col5
- K36 pad 2: /col5 -> /col6
- K37 pad 2: /col6 -> /col7
- K38 pad 2: /col7 -> /col8
- K39 pad 2: /col8 -> /col9
- K40 pad 2: /col9 -> /col10
- K41 pad 2: /col10 -> /col11
- K42 pad 2: /col11 -> /col12
- K43 pad 2: /col12 -> /col13
- K44 pad 2: /col13 -> /col14
- K45 pad 2: /col14 -> /col0
- K46 pad 2: /col0 -> /col1
- K47 pad 2: /col1 -> /col2
- K48 pad 2: /col2 -> /col3
- K49 pad 2: /col3 -> /col4
- K50 pad 2: /col4 -> /col5
- K51 pad 2: /col5 -> /col7
- K52 pad 2: /col7 -> /col9
- K53 pad 2: /col9 -> /col10
- K54 pad 2: /col10 -> /col11
- K55 pad 2: /col11 -> /col12
- K56 pad 2: /col12 -> /col13
- K57 pad 2: /col13 -> /col14
- K58 pad 2: /col14 -> /col0
- K59 pad 2: /col0 -> /col1
- K60 pad 2: /col1 -> /col2
- K61 pad 2: /col2 -> /col3
- K62 pad 2: /col3 -> /col4
- K63 pad 2: /col4 -> /col5
- K64 pad 2: /col5 -> /col6
- K65 pad 2: /col6 -> /col7
- K66 pad 2: /col7 -> /col8
- K67 pad 2: /col8 -> /col9
- K68 pad 2: /col9 -> /col10
- K69 pad 2: /col10 -> /col11
- K70 pad 2: /col11 -> /col12
- K71 pad 2: /col12 -> /col13
- K72 pad 2: /col13 -> /col14
- K73 pad 2: /col14 -> /col0
- K74 pad 2: /col0 -> /col1
- K75 pad 2: /col1 -> /col2
- K76 pad 2: /col2 -> /col3
- K77 pad 2: /col3 -> /col4
- K78 pad 2: /col4 -> /col5
- K79 pad 2: /col5 -> /col6
- K80 pad 2: /col6 -> /col8
- K81 pad 2: /col8 -> /col9
- K82 pad 2: /col9 -> /col10
- K83 pad 2: /col10 -> /col11
- K84 pad 2: /col11 -> /col12
- K85 pad 2: /col12 -> /col13
- K86 pad 2: /col13 -> /col14
Other:
- board outline added: 338.7 x 140.5 mm

Commit message: Updates
Parts:
- moved C1 57.2 mm to (158.0, 132.8), turned to 135 degrees
- moved C2 54.5 mm to (165.6, 125.2), turned to 135 degrees
- moved Y1 9.20 mm to (161.8, 129.0), turned to 90 degrees
- moved OLED1 4.74 mm to (200.0, 42.2)
- moved MCU1 3.66 mm to (172.0, 137.9), turned to 45 degrees
Routing:
- net /col6: track 0.00 -> 292.6 mm
- net /row2: track 0.00 -> 266.6 mm
- net /row1: track 0.00 -> 266.6 mm
- net /row0: track 0.00 -> 266.6 mm
- net /row4: track 0.00 -> 266.6 mm
- net /row5: track 0.00 -> 266.6 mm
- net /row3: track 0.00 -> 228.5 mm
- net /col7: track 0.00 -> 218.9 mm
- net /col14: track 0.00 -> 152.9 mm, vias 0 -> 1
- net /col8: track 0.00 -> 145.3 mm
- net /col13: track 0.00 -> 116.7 mm, vias 0 -> 1
- net /col12: track 0.00 -> 114.3 mm, vias 0 -> 1
- net /col11: track 0.00 -> 95.3 mm
- net /col9: track 0.00 -> 95.3 mm
- net /col5: track 0.00 -> 95.3 mm
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
Commit message: Updates
Routing:
- net /col0: track 95.2 -> 224.7 mm, vias 0 -> 1
- net /col1: track 95.2 -> 206.3 mm, vias 0 -> 1
- net /col2: track 95.3 -> 184.3 mm, vias 0 -> 1
- net /col13: track 116.7 -> 198.7 mm
- net /col3: track 95.3 -> 160.2 mm, vias 0 -> 1
- net /col14: track 152.9 -> 217.1 mm
- net /col12: track 114.3 -> 176.7 mm
- net /col11: track 95.3 -> 152.6 mm, vias 0 -> 1
- net /col4: track 95.3 -> 135.2 mm, vias 0 -> 1
- net /col10: track 95.3 -> 127.6 mm, vias 0 -> 1
- net VCC: track 0.00 -> 30.5 mm
- net /col5: track 95.3 -> 111.1 mm, vias 0 -> 1
- net /col9: track 95.3 -> 103.5 mm, vias 0 -> 1
