File: pcb/bloomer_v4.kicad_pcb (KiCad board)
At the start: 2 copper layers, 338.7 x 140.5 mm, 225 parts, among them K00 MX, K01 MX, K02 MX, K03 MX, K04 MX, K05 MX, K06 MX, K07 MX, K08 MX, K09 MX, K10 MX, K11 MX, K12 MX, K13 MX, K14 MX, K15 MX, K16 MX, K17 MX, K18 MX, K19 MX, K20 MX, K21 MX, K22 MX, K23 MX, K24 MX, K25 MX, K26 MX, K27 MX, K28 MX, K29 MX, K30 MX, K31 MX, K32 MX, K33 MX, K34 MX, K35 MX, K36 MX, K37 MX, K38 MX, K39 MX, K40 MX, K41 MX, K42 MX, K43 MX, K44 MX, K45 MX, K46 MX, K47 MX, K48 MX, K49 MX, K50 MX, K51 MX, K52 MX, K53 MX, K54 MX, K55 MX, K56 MX, K57 MX, K58 MX, K59 MX, K60 MX, K61 MX, K62 MX, K63 MX, K64 MX, K65 MX, K66 MX, K67 MX, K68 MX, K69 MX, K70 MX, K71 MX, K72 MX, K73 MX, K74 MX, K75 MX, K76 MX, K77 MX, K78 MX, K79 MX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

Commit message: Updates
Routing:
- net VCC: track 62.1 -> 700.1 mm, vias 0 -> 6
- net Net-(LED6-Pad2): track 0.00 -> 158.6 mm, vias 0 -> 2
- net Net-(LED10-Pad4): track 0.00 -> 81.9 mm, vias 0 -> 2
- net Net-(LED3-Pad2): track 6.34 -> 84.4 mm, vias 0 -> 2
- net Net-(LED5-Pad2): track 0.00 -> 39.4 mm
- net Net-(LED8-Pad2): track 0.00 -> 38.8 mm
- net Net-(LED10-Pad2): track 0.00 -> 38.1 mm
- net Net-(LED7-Pad2): track 0.00 -> 36.8 mm
- net Net-(LED11-Pad2): track 0.00 -> 36.6 mm
- net Net-(LED4-Pad2): track 0.00 -> 35.2 mm
- net Net-(LED2-Pad2): track 5.27 -> 35.2 mm
- net /row5: track 336.1 -> 344.8 mm, vias 0 -> 2
- net /row4: track 299.6 -> 307.5 mm, vias 0 -> 2
- net /row3: track 224.9 -> 232.1 mm, vias 0 -> 2
- net /row2: track 275.5 -> 282.0 mm, vias 0 -> 2
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- added copper zone on B.Cu, net (none)
- added copper zone on F.Cu, net GND

Commit message: Updates
Routing:
- net GND: track 0.00 -> 275.8 mm, vias 0 -> 22
- net /row4: track 307.5 -> 525.6 mm, vias 2 -> 4
- net /row3: track 232.1 -> 429.3 mm, vias 2 -> 3
- net /row2: track 282.0 -> 456.4 mm, vias 2 -> 3
- net /row1: track 318.4 -> 482.9 mm, vias 2 -> 3
- net VCC: track 700.1 -> 856.9 mm, vias 6 -> 10
- net /row0: track 354.3 -> 509.7 mm, vias 2 -> 3
- net /row5: track 344.8 -> 491.3 mm, vias 2 -> 3
- net /rgb: track 0.00 -> 133.7 mm, vias 0 -> 2
- net /usb_d-: track 0.00 -> 123.3 mm, vias 0 -> 2
- net /usb_d+: track 0.00 -> 119.0 mm, vias 0 -> 2
- net Net-(MCU1-Pad13): track 0.00 -> 98.0 mm, vias 0 -> 1
- net /col8: track 145.3 -> 234.0 mm, vias 0 -> 1
- net /col14: track 209.5 -> 293.0 mm, vias 2 -> 3
- net /col13: track 190.2 -> 272.2 mm, vias 2 -> 3
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- added copper zone on B.Cu, net GND
- removed copper zone on B.Cu, net (none)
Other:
- board text added: "Bloomer v4.0"
