File: pcb_test/bloomer.kicad_pcb (KiCad board)
At the start: 2 copper layers, 202 parts, among them J1 USB_mini_micro_B, K1 KEYSW, K10 KEYSW, K11 KEYSW, K12 KEYSW, K13 KEYSW, K14 KEYSW, K15 KEYSW, K16 KEYSW, K17 KEYSW, K18 KEYSW, K19 KEYSW, K2 KEYSW, K20 KEYSW, K21 KEYSW, K22 KEYSW, K23 KEYSW, K24 KEYSW, K25 KEYSW, K26 KEYSW, K27 KEYSW, K28 KEYSW, K29 KEYSW, K3 KEYSW, K30 KEYSW, K31 KEYSW, K32 KEYSW, K33 KEYSW, K34 KEYSW, K35 KEYSW, K36 KEYSW, K37 KEYSW, K38 KEYSW, K39 KEYSW, K4 KEYSW, K40 KEYSW, K41 KEYSW, K42 KEYSW, K43 KEYSW, K44 KEYSW, K45 KEYSW, K46 KEYSW, K47 KEYSW, K48 KEYSW, K49 KEYSW, K5 KEYSW, K50 KEYSW, K51 KEYSW, K52 KEYSW, K53 KEYSW, K54 KEYSW, K55 KEYSW, K56 KEYSW, K57 KEYSW, K58 KEYSW, K59 KEYSW, K6 KEYSW, K60 KEYSW, K61 KEYSW, K62 KEYSW, K63 KEYSW, K64 KEYSW, K65 KEYSW, K66 KEYSW, K67 KEYSW, K68 KEYSW, K69 KEYSW, K7 KEYSW, K70 KEYSW, K71 KEYSW, K72 KEYSW, K73 KEYSW, K74 KEYSW, K75 KEYSW, K76 KEYSW, K77 KEYSW, K78 KEYSW, K79 KEYSW, K8 KEYSW, K80 KEYSW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

Commit message: Updaes
Parts:
- moved L4 224.9 mm to (321.1, 113.4), turned to 10 degrees
- moved L9 194.1 mm to (48.9, 113.4), turned to -10 degrees
- moved L3 187.2 mm to (307.8, 38.3), turned to 190 degrees
- moved L5 186.9 mm to (282.2, 112.1), turned to 10 degrees
- moved L6 172.8 mm to (246.6, 129.6), turned to 10 degrees
- moved L8 161.1 mm to (87.8, 112.1), turned to -10 degrees
- moved L2 159.5 mm to (268.9, 37.1), turned to 190 degrees
- moved L7 156.6 mm to (123.5, 129.6), turned to -10 degrees
- moved L10 149.7 mm to (62.2, 38.3), turned to -190 degrees
- moved L1 144.1 mm to (233.3, 54.5), turned to 190 degrees
- moved L12 124.7 mm to (136.7, 54.5), turned to -190 degrees
- moved L11 93.7 mm to (101.1, 37.1), turned to -190 degrees
Changed lines of the file:
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@@
   )
   (module LED_SMD:LED_WS2812B_PLCC4_5.0x5.0mm_P3.2mm (layer B.Cu)
-    (at 110 -20)
+    (at 233.318 54.511 190)
     (descr https://cdn-shop.adafruit.com/datasheets/WS2812B.pdf)
     (tags "LED RGB NeoPixel")
@@
   )
   (module LED_SMD:LED_WS2812B_PLCC4_5.0x5.0mm_P3.2mm (layer B.Cu)
-    (at 120 -20)
+    (at 268.929 37.062 190)
     (descr https://cdn-shop.adafruit.com/datasheets/WS2812B.pdf)
     (tags "LED RGB NeoPixel")
@@
   )
   (module LED_SMD:LED_WS2812B_PLCC4_5.0x5.0mm_P3.2mm (layer B.Cu)
-    (at 130 -20)
+    (at 307.839 38.325 190)
     (descr https://cdn-shop.adafruit.com/datasheets/WS2812B.pdf)
     (tags "LED RGB NeoPixel")
@@
   )
   (module LED_SMD:LED_WS2812B_PLCC4_5.0x5.0mm_P3.2mm (layer B.Cu)
-    (at 140 -20)
+    (at 321.071 113.367 10)
     (descr https://cdn-shop.adafruit.com/datasheets/WS2812B.pdf)
     (tags "LED RGB NeoPixel")
@@
   )
   (module LED_SMD:LED_WS2812B_PLCC4_5.0x5.0mm_P3.2mm (layer B.Cu)
-    (at 150 -20)
+    (at 282.161 112.105 10)
     (descr https://cdn-shop.adafruit.com/datasheets/WS2812B.pdf)
     (tags "LED RGB NeoPixel")
@@
   )
   (module LED_SMD:LED_WS2812B_PLCC4_5.0x5.0mm_P3.2mm (layer B.Cu)
-    (at 160 -20)
+    (at 246.55 129.553 10)
     (descr https://cdn-shop.adafruit.com/datasheets/WS2812B.pdf)
     (tags "LED RGB NeoPixel")
@@
   )
   (module LED_SMD:LED_WS2812B_PLCC4_5.0x5.0mm_P3.2mm (layer B.Cu)
-    (at 170 -20)
+    (at 123.45 129.553 -10)
     (descr https://cdn-shop.adafruit.com/datasheets/WS2812B.pdf)
     (tags "LED RGB NeoPixel")
@@
   )
   (module LED_SMD:LED_WS2812B_PLCC4_5.0x5.0mm_P3.2mm (layer B.Cu)
-    (at 180 -20)
+    (at 87.839 112.105 -10)
     (descr https://cdn-shop.adafruit.com/datasheets/WS2812B.pdf)
     (tags "LED RGB NeoPixel")
@@
   )
   (module LED_SMD:LED_WS2812B_PLCC4_5.0x5.0mm_P3.2mm (layer B.Cu)
-    (at 190 -20)
+    (at 48.929 113.367 -10)
     (descr https://cdn-shop.adafruit.com/datasheets/WS2812B.pdf)
     (tags "LED RGB NeoPixel")
@@
   )
   (module LED_SMD:LED_WS2812B_PLCC4_5.0x5.0mm_P3.2mm (layer B.Cu)
-    (at 200 -20)
+    (at 62.161 38.325 -190)
     (descr https://cdn-shop.adafruit.com/datasheets/WS2812B.pdf)
     (tags "LED RGB NeoPixel")
@@
   )
   (module LED_SMD:LED_WS2812B_PLCC4_5.0x5.0mm_P3.2mm (layer B.Cu)
-    (at 20 -10)
+    (at 101.071 37.062 -190)
     (descr https://cdn-shop.adafruit.com/datasheets/WS2812B.pdf)
     (tags "LED RGB NeoPixel")
@@
   )
   (module LED_SMD:LED_WS2812B_PLCC4_5.0x5.0mm_P3.2mm (layer B.Cu)
-    (at 30 -10)
-    (descr https://cdn-shop.adafruit.com/datasheets/WS2812B.pdf)
-    (tags "LED RGB NeoPixel")
+    (at 136.682 54.511 -190)
+    (descr https://cdn-shop.adafruit.com/datasheets/WS2812B.pdf)
+    (tags "LED RGB NeoPixel")

Commit message: Updates
Parts:
- moved C3 215.4 mm to (204.5, 119.1), turned to 90 degrees
- moved C4 211.1 mm to (208.9, 119.0), turned to 90 degrees
- moved C5 207.0 mm to (213.4, 119.1), turned to 90 degrees
- moved C6 202.9 mm to (217.8, 119.1), turned to 90 degrees
- moved C7 198.9 mm to (222.2, 119.1), turned to 90 degrees
- moved C2 180.4 mm to (154.3, 110.7), turned to 270 degrees
- moved C1 179.4 mm to (142.9, 110.7), turned to 270 degrees
- moved R2 178.0 mm to (163.2, 127.4), turned to 90 degrees
- moved R1 172.9 mm to (163.2, 111.4), turned to 270 degrees
- moved C8 151.0 mm to (139.1, 122.8), turned to 270 degrees
- moved U1 145.5 mm to (148.6, 123.2)
- moved X1 130.0 mm to (148.4, 110.6)
- moved SW1 128.5 mm to (185.4, 63.5)
- moved R3 121.4 mm to (172.1, 36.6), turned to 90 degrees
- moved R4 116.4 mm to (176.7, 36.6), turned to 90 degrees
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- renumbered D41 to D40, D40 to D41, D51 to D50, D50 to D51, K41 to K40, K40 to K41, K51 to K50, K50 to K51
Connections:
- D40 pad 1: /row5 -> /row4
- D41 pad 1: /row4 -> /row5
- D50 pad 1: /row5 -> /row4
- D51 pad 1: /row4 -> /row5
