File: pcb_test/bloomer.kicad_pcb (KiCad board)
At the start: 2 copper layers, 202 parts, among them J1 USB_mini_micro_B, K1 KEYSW, K10 KEYSW, K11 KEYSW, K12 KEYSW, K13 KEYSW, K14 KEYSW, K15 KEYSW, K16 KEYSW, K17 KEYSW, K18 KEYSW, K19 KEYSW, K2 KEYSW, K20 KEYSW, K21 KEYSW, K22 KEYSW, K23 KEYSW, K24 KEYSW, K25 KEYSW, K26 KEYSW, K27 KEYSW, K28 KEYSW, K29 KEYSW, K3 KEYSW, K30 KEYSW, K31 KEYSW, K32 KEYSW, K33 KEYSW, K34 KEYSW, K35 KEYSW, K36 KEYSW, K37 KEYSW, K38 KEYSW, K39 KEYSW, K4 KEYSW, K40 KEYSW, K41 KEYSW, K42 KEYSW, K43 KEYSW, K44 KEYSW, K45 KEYSW, K46 KEYSW, K47 KEYSW, K48 KEYSW, K49 KEYSW, K5 KEYSW, K50 KEYSW, K51 KEYSW, K52 KEYSW, K53 KEYSW, K54 KEYSW, K55 KEYSW, K56 KEYSW, K57 KEYSW, K58 KEYSW, K59 KEYSW, K6 KEYSW, K60 KEYSW, K61 KEYSW, K62 KEYSW, K63 KEYSW, K64 KEYSW, K65 KEYSW, K66 KEYSW, K67 KEYSW, K68 KEYSW, K69 KEYSW, K7 KEYSW, K70 KEYSW, K71 KEYSW, K72 KEYSW, K73 KEYSW, K74 KEYSW, K75 KEYSW, K76 KEYSW, K77 KEYSW, K78 KEYSW, K79 KEYSW, K8 KEYSW, K80 KEYSW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

Commit message: Updates
Parts:
- removed X1: XTAL_GND, Crystal:Crystal_SMD_TXC_7M-4Pin_3.2x2.5mm_HandSoldering
- added Y1: Crystal_GND24, Crystal:Crystal_SMD_TXC_7M-4Pin_3.2x2.5mm_HandSoldering, B.Cu at (154.0, 8.76)
- moved C6 75.2 mm to (142.9, 27.6)
- moved C7 73.4 mm to (149.5, 30.5), turned to 0 degrees
- moved C3 59.1 mm to (146.1, 11.7)
- moved C5 54.6 mm to (159.6, 30.5), turned to 180 degrees
- moved C4 43.3 mm to (165.7, 17.4)
- moved D40 25.5 mm to (148.4, 143.6), turned to 80 degrees
- moved D41 25.5 mm to (173.9, 144.1), turned to 90 degrees
- moved D50 25.5 mm to (237.3, 140.9), turned to 100 degrees
- moved D51 25.5 mm to (212.1, 144.1), turned to 90 degrees
- moved K40 25.5 mm to (140.6, 142.2), turned to 350 degrees
- moved K41 25.5 mm to (165.9, 144.1), turned to 0 degrees
- moved K50 25.5 mm to (229.4, 142.2), turned to 10 degrees
- moved K51 25.5 mm to (204.1, 144.1), turned to 0 degrees
- moved R1 18.9 mm to (144.4, 15.2), turned to 180 degrees
- moved R4 15.7 mm to (192.4, 36.0), turned to 270 degrees
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- renumbered D41 to D40, D40 to D41, D51 to D50, D50 to D51, K41 to K40, K40 to K41, K51 to K50, K50 to K51
Connections:
- net +5V renamed GND
- D40 pad 1: /row5 -> /row4
- D41 pad 1: /row4 -> /row5
- D50 pad 1: /row5 -> /row4
- D51 pad 1: /row4 -> /row5
- K82 pad 1: Net-(K82-Pad1) -> /col14
- K83 pad 1: Net-(K82-Pad1) -> /col14
- K84 pad 1: Net-(K82-Pad1) -> /col14
- K85 pad 1: Net-(K82-Pad1) -> /col14
- K86 pad 1: Net-(K82-Pad1) -> /col14
- K87 pad 1: Net-(K82-Pad1) -> /col14
Routing:
- net /row0: track 0.00 -> 242.3 mm
- net /row2: track 0.00 -> 242.3 mm
- net /row5: track 0.00 -> 242.3 mm
- net /row1: track 0.00 -> 242.3 mm
- net /col0: track 0.00 -> 210.7 mm, vias 0 -> 1
- net /row4: track 0.00 -> 204.2 mm
- net /row3: track 0.00 -> 204.2 mm
- net /col14: track 0.00 -> 204.2 mm, vias 0 -> 1
- net /col1: track 0.00 -> 191.6 mm, vias 0 -> 1
- net /col13: track 0.00 -> 185.1 mm, vias 0 -> 1
- net /col2: track 0.00 -> 171.5 mm, vias 0 -> 1
- net /col12: track 0.00 -> 167.8 mm, vias 0 -> 1
- net /col3: track 0.00 -> 150.0 mm, vias 0 -> 1
- net /col11: track 0.00 -> 147.4 mm, vias 0 -> 1
- net /col4: track 0.00 -> 127.7 mm, vias 0 -> 1
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
Commit message: Updates
Routing:
- net Net-(U1-Pad11): track 0.00 -> 204.2 mm, vias 0 -> 1
- net /col14: track 204.2 -> 0.00 mm, vias 1 -> 0
- net GND: track 88.4 -> 0.00 mm, vias 3 -> 0
- net VCC: track 60.7 -> 0.00 mm, vias 3 -> 0
- net /col5: track 106.1 -> 145.7 mm
- net /col4: track 127.7 -> 166.2 mm
- net /col3: track 150.0 -> 187.5 mm
- net /col2: track 171.5 -> 195.6 mm
- net /col1: track 191.6 -> 214.7 mm
- net /col0: track 210.7 -> 232.7 mm
- net Net-(C1-Pad1): track 14.7 -> 0.00 mm
- net Net-(C2-Pad1): track 10.4 -> 0.00 mm
- net /col8: track 102.3 -> 95.2 mm
- net Net-(R1-Pad1): track 7.07 -> 0.00 mm
- net Net-(C8-Pad1): track 6.05 -> 0.00 mm
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
Commit message: Updates
Parts:
- moved C2 122.0 mm to (152.7, 131.1), turned to 135 degrees
- moved Y1 119.7 mm to (155.9, 128.4), turned to 225 degrees
- moved C1 116.4 mm to (158.5, 125.2), turned to 135 degrees
- moved C3 115.1 mm to (163.2, 125.5), turned to 270 degrees
- moved R1 108.6 mm to (164.9, 121.9), turned to 0 degrees
- moved C4 104.8 mm to (143.5, 119.8), turned to 270 degrees
- moved C8 96.4 mm to (166.4, 115.3), turned to 90 degrees
- moved U1 94.0 mm to (154.9, 115.6), turned to 180 degrees
- moved C6 85.4 mm to (166.4, 109.6), turned to 270 degrees
- moved R2 84.5 mm to (146.7, 110.1), turned to 270 degrees
- moved C7 76.9 mm to (159.8, 106.7), turned to 180 degrees
- moved C5 76.9 mm to (149.6, 106.7), turned to 0 degrees
- moved R3 1.49 mm to (178.7, 36.0)
- moved R4 1.06 mm to (191.3, 36.0)
- moved SW1 0.32 mm to (185.0, 63.2)
Routing:
- net /col14: track 0.00 -> 301.2 mm, vias 0 -> 3
- net /row4: track 204.2 -> 431.7 mm, vias 0 -> 7
- net Net-(U1-Pad11): track 204.2 -> 0.00 mm, vias 1 -> 0
- net /row5: track 242.3 -> 403.3 mm, vias 0 -> 4
- net /col9: track 99.6 -> 251.9 mm
- net /col10: track 121.1 -> 273.3 mm
- net /col11: track 143.5 -> 295.3 mm
- net /col12: track 165.0 -> 304.1 mm
- net /row3: track 204.2 -> 332.3 mm, vias 0 -> 5
- net /col13: track 185.1 -> 281.4 mm, vias 1 -> 3
- net /col8: track 95.2 -> 188.6 mm, vias 0 -> 1
- net /row0: track 242.3 -> 328.9 mm, vias 0 -> 2
- net GND: track 0.00 -> 78.5 mm, vias 0 -> 5
- net /row1: track 242.3 -> 313.2 mm, vias 0 -> 2
- net VCC: track 0.00 -> 68.3 mm
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