File: pcb_test/bloomer.test.kicad_pcb (KiCad board)
At the start: 2 copper layers, 202 parts, among them J1 USB_mini_micro_B, K1 KEYSW, K10 KEYSW, K11 KEYSW, K12 KEYSW, K13 KEYSW, K14 KEYSW, K15 KEYSW, K16 KEYSW, K17 KEYSW, K18 KEYSW, K19 KEYSW, K2 KEYSW, K20 KEYSW, K21 KEYSW, K22 KEYSW, K23 KEYSW, K24 KEYSW, K25 KEYSW, K26 KEYSW, K27 KEYSW, K28 KEYSW, K29 KEYSW, K3 KEYSW, K30 KEYSW, K31 KEYSW, K32 KEYSW, K33 KEYSW, K34 KEYSW, K35 KEYSW, K36 KEYSW, K37 KEYSW, K38 KEYSW, K39 KEYSW, K4 KEYSW, K40 KEYSW, K41 KEYSW, K42 KEYSW, K43 KEYSW, K44 KEYSW, K45 KEYSW, K46 KEYSW, K47 KEYSW, K48 KEYSW, K49 KEYSW, K5 KEYSW, K50 KEYSW, K51 KEYSW, K52 KEYSW, K53 KEYSW, K54 KEYSW, K55 KEYSW, K56 KEYSW, K57 KEYSW, K58 KEYSW, K59 KEYSW, K6 KEYSW, K60 KEYSW, K61 KEYSW, K62 KEYSW, K63 KEYSW, K64 KEYSW, K65 KEYSW, K66 KEYSW, K67 KEYSW, K68 KEYSW, K69 KEYSW, K7 KEYSW, K70 KEYSW, K71 KEYSW, K72 KEYSW, K73 KEYSW, K74 KEYSW, K75 KEYSW, K76 KEYSW, K77 KEYSW, K78 KEYSW, K79 KEYSW, K8 KEYSW, K80 KEYSW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

Commit message: Updates
Parts:
- moved C6 76.4 mm to (141.6, 26.3)
- moved C7 74.5 mm to (148.2, 29.2), turned to 0 degrees
- moved C3 60.6 mm to (144.8, 10.4)
- moved C5 55.7 mm to (158.4, 29.2), turned to 180 degrees
- moved C4 44.7 mm to (164.5, 16.1)
- moved R1 20.5 mm to (143.1, 13.3), turned to 180 degrees
- moved R4 15.7 mm to (192.4, 36.0), turned to 270 degrees
- moved C1 10.6 mm to (148.6, 7.87)
- moved X1 9.94 mm to (152.9, 7.74)
- moved C2 9.25 mm to (156.8, 7.87)
- moved C8 8.40 mm to (141.6, 20.6)
- moved U1 8.25 mm to (153.0, 20.3)
- moved R3 5.12 mm to (177.2, 36.0), turned to 270 degrees
- moved R2 3.77 mm to (161.3, 25.8)
Connections:
- C1 pad 2: +5V -> GND
- C2 pad 2: +5V -> GND
- C3 pad 2: +5V -> GND
- C4 pad 2: +5V -> GND
- C5 pad 2: +5V -> GND
- C6 pad 2: +5V -> GND
- C7 pad 2: +5V -> GND
- C8 pad 2: +5V -> GND
- J1 pad 5: +5V -> GND
- J1 pad 6: +5V -> GND
- K82 pad 1: Net-(K82-Pad1) -> /col14
- K83 pad 1: Net-(K82-Pad1) -> /col14
- K84 pad 1: Net-(K82-Pad1) -> /col14
- K85 pad 1: Net-(K82-Pad1) -> /col14
- K86 pad 1: Net-(K82-Pad1) -> /col14
- K87 pad 1: Net-(K82-Pad1) -> /col14
- L1 pad 3: +5V -> GND
- L10 pad 3: +5V -> GND
- L11 pad 3: +5V -> GND
- L12 pad 3: +5V -> GND
- L2 pad 3: +5V -> GND
- L3 pad 3: +5V -> GND
- L4 pad 3: +5V -> GND
- L5 pad 3: +5V -> GND
- L6 pad 3: +5V -> GND
- L7 pad 3: +5V -> GND
- L8 pad 3: +5V -> GND
- L9 pad 3: +5V -> GND
- R2 pad 1: +5V -> GND
- SW1 pad 1: +5V -> GND
- U1 pad 15: +5V -> GND
- U1 pad 23: +5V -> GND
- U1 pad 35: +5V -> GND
- U1 pad 43: +5V -> GND
- U1 pad 5: +5V -> GND
- X1 pad 3: +5V -> GND
- X1 pad 4: (no net) -> GND
Routing:
- net /row0: track 0.00 -> 242.3 mm
- net /row2: track 0.00 -> 242.3 mm
- net /row5: track 0.00 -> 242.3 mm
- net /row1: track 0.00 -> 242.3 mm
- net /col0: track 0.00 -> 210.7 mm, vias 0 -> 1
- net /row4: track 0.00 -> 204.2 mm
- net /row3: track 0.00 -> 204.2 mm
- net /col14: track 0.00 -> 204.2 mm, vias 0 -> 1
- net /col1: track 0.00 -> 191.6 mm, vias 0 -> 1
- net /col13: track 0.00 -> 185.1 mm, vias 0 -> 1
- net /col2: track 0.00 -> 171.5 mm, vias 0 -> 1
- net /col12: track 0.00 -> 167.8 mm, vias 0 -> 1
- net /col3: track 0.00 -> 150.0 mm, vias 0 -> 1
- net /col11: track 0.00 -> 147.4 mm, vias 0 -> 1
- net /col4: track 0.00 -> 127.7 mm, vias 0 -> 1
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